File: KiCad Files/RowdyTestBoard2.kicad_sch (KiCad schematic)
At the start: 0 parts

Commit message: Coils done
Other:
- sheet Coils ports: added 5V, Data Serial, NMR, NOE, QH', SHCP, STCP; removed none
Changed lines of the file:
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@@
       (effects (font (size 1.27 1.27)) (justify left top))
+    )
+    (pin "QH'" input (at 103.886 76.2 0)
+      (effects (font (size 1.27 1.27)) (justify right))
+    )
+    (pin "Data Serial" input (at 103.886 42.164 0)
+      (effects (font (size 1.27 1.27)) (justify right))
+    )
+    (pin "NOE" input (at 103.886 45.212 0)
+      (effects (font (size 1.27 1.27)) (justify right))
+    )
+    (pin "SHCP" input (at 103.886 48.514 0)
+      (effects (font (size 1.27 1.27)) (justify right))
+    )
+    (pin "STCP" input (at 103.886 51.562 0)
+      (effects (font (size 1.27 1.27)) (justify right))
+    )
+    (pin "NMR" input (at 103.886 73.406 0)
+      (effects (font (size 1.27 1.27)) (justify right))
+    )
+    (pin "5V" input (at 103.886 39.116 0)
+      (effects (font (size 1.27 1.27)) (justify right))
     )
   )

Commit message: hello
Parts:
- added J? (x2): Conn_02x04_Odd_Even, Connector_PinSocket_2.54mm:PinSocket_2x04_P2.54mm_Vertical_SMD, symbol Connector_Generic:Conn_02x04_Odd_Even
Changed lines of the file:
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@@
 (kicad_sch (version 20211123) (generator eeschema)
   (paper "A4")
+  (symbol (lib_id "Connector_Generic:Conn_02x04_Odd_Even") (at 226.06 73.66 0) (unit 1)
+    (in_bom yes) (on_board yes) (fields_autoplaced)
+    (property "Reference" "J?" (id 0) (at 227.33 64.6938 0))
+    (property "Value" "Conn_02x04_Odd_Even" (id 1) (at 227.33 67.2338 0))
+    (property "Footprint" "Connector_PinSocket_2.54mm:PinSocket_2x04_P2.54mm_Vertical_SMD" (id 2) (at 226.06 73.66 0)
+      (effects (font (size 1.27 1.27)) hide)
+    )
+    (property "Datasheet" "https://datasheet.lcsc.com/lcsc/2108131730_BOOMELE-Boom-Precision-Elec-C192300_C192300.pdf" (id 3) (at 226.06 73.66 0)
+      (effects (font (size 1.27 1.27)) hide)
+    )
+    (pin "1")
+    (pin "2")
+    (pin "3")
+    (pin "4")
+    (pin "5")
+    (pin "6")
+    (pin "7")
+    (pin "8")
+  )
+  (symbol (lib_id "Connector_Generic:Conn_02x04_Odd_Even") (at 226.06 53.34 0) (unit 1)
+    (in_bom yes) (on_board yes) (fields_autoplaced)
+    (property "Reference" "J?" (id 0) (at 227.33 44.3738 0))
+    (property "Value" "Conn_02x04_Odd_Even" (id 1) (at 227.33 46.9138 0))
+    (property "Footprint" "Connector_PinSocket_2.54mm:PinSocket_2x04_P2.54mm_Vertical_SMD" (id 2) (at 226.06 53.34 0)
+      (effects (font (size 1.27 1.27)) hide)
+    )
+    (property "Datasheet" "https://datasheet.lcsc.com/lcsc/2108131730_BOOMELE-Boom-Precision-Elec-C192300_C192300.pdf" (id 3) (at 226.06 53.34 0)
+      (effects (font (size 1.27 1.27)) hide)
+    )
+    (pin "1")
+    (pin "2")
+    (pin "3")
+    (pin "4")
+    (pin "5")
+    (pin "6")
+    (pin "7")
+    (pin "8")
+  )
   (sheet (at 38.354 99.314) (size 65.278 48.006) (fields_autoplaced)
     (stroke (width 0.1524) (type solid) (color 0 0 0 0))
@@
       (reference "#PWR?") (unit 1) (value "GND") (footprint "")
     )
+    (path "/8e79823e-4332-4e10-8228-ec68b8b05a31"
+      (reference "J?") (unit 1) (value "Conn_02x04_Odd_Even") (footprint "Connector_PinSocket_2.54mm:PinSocket_2x04_P2.54mm_Vertical_SMD")
+    )
+    (path "/be78c320-66c9-47db-84c6-e07682b2c3ee"
+      (reference "J?") (unit 1) (value "Conn_02x04_Odd_Even") (footprint "Connector_PinSocket_2.54mm:PinSocket_2x04_P2.54mm_Vertical_SMD")
+    )
     (path "/590c1e64-bea6-4659-9fa3-7b726d55c0d8/2beb55be-3789-42e2-a70f-e1828b5d435c"

Commit message: hall1
Parts:
- removed J? (x2): Conn_02x04_Odd_Even, Connector_PinSocket_2.54mm:PinSocket_2x04_P2.54mm_Vertical_SMD, symbol Connector_Generic:Conn_02x04_Odd_Even
Changed lines of the file:
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@@
 (kicad_sch (version 20211123) (generator eeschema)
   (paper "A4")
-  (symbol (lib_id "Connector_Generic:Conn_02x04_Odd_Even") (at 226.06 73.66 0) (unit 1)
-    (in_bom yes) (on_board yes) (fields_autoplaced)
-    (property "Reference" "J?" (id 0) (at 227.33 64.6938 0))
-    (property "Value" "Conn_02x04_Odd_Even" (id 1) (at 227.33 67.2338 0))
-    (property "Footprint" "Connector_PinSocket_2.54mm:PinSocket_2x04_P2.54mm_Vertical_SMD" (id 2) (at 226.06 73.66 0)
-      (effects (font (size 1.27 1.27)) hide)
-    )
-    (property "Datasheet" "https://datasheet.lcsc.com/lcsc/2108131730_BOOMELE-Boom-Precision-Elec-C192300_C192300.pdf" (id 3) (at 226.06 73.66 0)
-      (effects (font (size 1.27 1.27)) hide)
-    )
-    (pin "1")
-    (pin "2")
-    (pin "3")
-    (pin "4")
-    (pin "5")
-    (pin "6")
-    (pin "7")
-    (pin "8")
-  )
-  (symbol (lib_id "Connector_Generic:Conn_02x04_Odd_Even") (at 226.06 53.34 0) (unit 1)
-    (in_bom yes) (on_board yes) (fields_autoplaced)
-    (property "Reference" "J?" (id 0) (at 227.33 44.3738 0))
-    (property "Value" "Conn_02x04_Odd_Even" (id 1) (at 227.33 46.9138 0))
-    (property "Footprint" "Connector_PinSocket_2.54mm:PinSocket_2x04_P2.54mm_Vertical_SMD" (id 2) (at 226.06 53.34 0)
-      (effects (font (size 1.27 1.27)) hide)
-    )
-    (property "Datasheet" "https://datasheet.lcsc.com/lcsc/2108131730_BOOMELE-Boom-Precision-Elec-C192300_C192300.pdf" (id 3) (at 226.06 53.34 0)
-      (effects (font (size 1.27 1.27)) hide)
-    )
-    (pin "1")
-    (pin "2")
-    (pin "3")
-    (pin "4")
-    (pin "5")
-    (pin "6")
-    (pin "7")
-    (pin "8")
-  )
   (sheet (at 38.354 99.314) (size 65.278 48.006) (fields_autoplaced)
     (stroke (width 0.1524) (type solid) (color 0 0 0 0))
@@
       (reference "#PWR04") (unit 1) (value "GND") (footprint "")
     )
+    (path "/a6b1e09a-8af3-4cc4-9df1-f67a0e8f20fc/90bfdf0e-1491-4904-8db8-cf5e40170b4e"
+      (reference "#PWR?") (unit 1) (value "GND") (footprint "")
+    )
+    (path "/a6b1e09a-8af3-4cc4-9df1-f67a0e8f20fc/b3a211ab-cde8-4082-b259-f7f4a4cc663f"
+      (reference "#PWR?") (unit 1) (value "GND") (footprint "")
+    )
+    (path "/a6b1e09a-8af3-4cc4-9df1-f67a0e8f20fc/c873ee13-bc72-41e5-a1ae-57ece8d4a9f5"
+      (reference "#PWR?") (unit 1) (value "GND") (footprint "")
+    )
     (path "/590c1e64-bea6-4659-9fa3-7b726d55c0d8/cdb9a0e2-cf2e-4003-b5c9-8bddb9e96904"
       (reference "#PWR?") (unit 1) (value "GND") (footprint "")
     )
-    (path "/8e79823e-4332-4e10-8228-ec68b8b05a31"
-      (reference "J?") (unit 1) (value "Conn_02x04_Odd_Even") (footprint "Connector_PinSocket_2.54mm:PinSocket_2x04_P2.54mm_Vertical_SMD")
+    (path "/a6b1e09a-8af3-4cc4-9df1-f67a0e8f20fc/fcf7c376-905e-4f32-a487-bc8568d498bd"
+      (reference "#PWR?") (unit 1) (value "GND") (footprint "")
     )
-    (path "/be78c320-66c9-47db-84c6-e07682b2c3ee"
-      (reference "J?") (unit 1) (value "Conn_02x04_Odd_Even") (footprint "Connector_PinSocket_2.54mm:PinSocket_2x04_P2.54mm_Vertical_SMD")
+    (path "/a6b1e09a-8af3-4cc4-9df1-f67a0e8f20fc/266b7e6f-426b-43f7-b46d-50ac4ff256b9"
+      (reference "IC?") (unit 1) (value "AH1902-Z-7") (footprint "AH1902Z7")
+    )
+    (path "/a6b1e09a-8af3-4cc4-9df1-f67a0e8f20fc/7b3f904b-56d8-43af-af24-37ea6851b116"
+      (reference "IC?") (unit 1) (value "AH1902-Z-7") (footprint "AH1902Z7")
+    )
+    (path "/a6b1e09a-8af3-4cc4-9df1-f67a0e8f20fc/94b7b858-992d-497a-bd6b-051f4dea2255"
+      (reference "IC?") (unit 1) (value "AH1902-Z-7") (footprint "AH1902Z7")
+    )
+    (path "/a6b1e09a-8af3-4cc4-9df1-f67a0e8f20fc/ff45e544-680d-4099-bd07-451c5137b60b"
+      (reference "IC?") (unit 1) (value "AH1902-Z-7") (footprint "AH1902Z7")
     )
     (path "/590c1e64-bea6-4659-9fa3-7b726d55c0d8/2beb55be-3789-42e2-a70f-e1828b5d435c"

Commit message: Startpcb
Other:
- sheet Sensors ports: added 3V, 5V, ClkEnIn, ClkIn, NPL, NSEROutput, SEROutput; removed none
Changed lines of the file:
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@@
       (effects (font (size 1.27 1.27)) (justify left top))
+    )
+    (pin "NSEROutput" input (at 204.724 49.53 0)
+      (effects (font (size 1.27 1.27)) (justify right))
+    )
+    (pin "SEROutput" input (at 204.724 52.832 0)
+      (effects (font (size 1.27 1.27)) (justify right))
+    )
+    (pin "5V" input (at 204.724 38.608 0)
+      (effects (font (size 1.27 1.27)) (justify right))
+    )
+    (pin "3V" input (at 204.724 41.656 0)
+      (effects (font (size 1.27 1.27)) (justify right))
+    )
+    (pin "NPL" input (at 204.724 55.88 0)
+      (effects (font (size 1.27 1.27)) (justify right))
+    )
+    (pin "ClkEnIn" input (at 204.724 58.928 0)
+      (effects (font (size 1.27 1.27)) (justify right))
+    )
+    (pin "ClkIn" input (at 204.724 61.722 0)
+      (effects (font (size 1.27 1.27)) (justify right))
     )
   )
