File: KiCad Files/RowdyTestBoard2.kicad_sch (KiCad schematic)
At the start: 0 parts

Commit message: Pcb2
Parts:
- added D1: 1N5819, Diode_THT:D_DO-41_SOD81_P10.16mm_Horizontal, symbol Diode:1N5819
- added J1, J2: Conn_02x04_Top_Bottom, Connector_PinHeader_2.54mm:PinHeader_2x04_P2.54mm_Vertical_SMD, symbol Connector_Generic:Conn_02x04_Top_Bottom
- added U1: USB-C, USB_C:USB-C-SMD_KH-TYPE-C-16P, symbol usb-c:USB-C
Connections:
- new net: D1.2 (A), U1.A4 (VBUS), U1.A9 (VBUS), U1.B4 (VBUS), U1.B9 (VBUS)
- new net 3V: J1.1 (Pin_1)
- new net ClkEnIn: J1.6 (Pin_6)
- new net ClkIn: J1.5 (Pin_5)
- new net Data Serial: J2.5 (Pin_5)
- new net GND: U1.A1 (GND), U1.A12 (GND), U1.A5 (CC1), U1.A6 (DP1), U1.A7 (DN1), U1.A8 (SUB1), U1.B1 (GND), U1.B12 (GND), U1.B5 (CC2), U1.B6 (DP2), U1.B7 (DN2), U1.B8 (SUB2)
- new net NMR: J2.1 (Pin_1)
- new net NOE: J2.6 (Pin_6)
- new net NPL: J1.7 (Pin_7)
- new net NSEROutput: J1.4 (Pin_4)
- new net QH': J2.2 (Pin_2)
- new net SEROutput: J1.8 (Pin_8)
- new net SHCP: J2.7 (Pin_7)
- new net STCP: J2.8 (Pin_8)
- new net VBus: D1.1 (K)
Other:
- removed sheet Microcontroller
- removed sheet Power

Commit message: diode
Parts:
- D1: footprint Diode_THT:D_DO-41_SOD81_P10.16mm_Horizontal -> Diode_SMD:D_SOD-323F; JLC Part Number (none) -> C2128
Changed lines of the file:
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@@
     (property "Reference" "D1" (id 0) (at 102.4255 115.824 0))
     (property "Value" "1N5819" (id 1) (at 102.4255 118.364 0))
-    (property "Footprint" "Diode_THT:D_DO-41_SOD81_P10.16mm_Horizontal" (id 2) (at 102.108 118.237 0)
+    (property "Footprint" "Diode_SMD:D_SOD-323F" (id 2) (at 102.108 118.237 0)
       (effects (font (size 1.27 1.27)) hide)
     )
     (property "Datasheet" "http://www.vishay.com/docs/88525/1n5817.pdf" (id 3) (at 102.108 122.682 0)
+      (effects (font (size 1.27 1.27)) hide)
+    )
+    (property "JLC Part Number" "C2128" (id 4) (at 102.108 122.682 0)
       (effects (font (size 1.27 1.27)) hide)
     )
@@
     )
     (path "/06df2c7b-9992-4fe2-8804-c49a5197fa1a"
-      (reference "D1") (unit 1) (value "1N5819") (footprint "Diode_THT:D_DO-41_SOD81_P10.16mm_Horizontal")
+      (reference "D1") (unit 1) (value "1N5819") (footprint "Diode_SMD:D_SOD-323F")
     )
     (path "/a6b1e09a-8af3-4cc4-9df1-f67a0e8f20fc/ff45e544-680d-4099-bd07-451c5137b60b"
-      (reference "IC1") (unit 1) (value "AH1902-Z-7") (footprint "AH1902Z7")
+      (reference "IC1") (unit 1) (value "AH1902-Z-7") (footprint "HallSensor:AH1902Z7")
     )
     (path "/a6b1e09a-8af3-4cc4-9df1-f67a0e8f20fc/266b7e6f-426b-43f7-b46d-50ac4ff256b9"
-      (reference "IC2") (unit 1) (value "AH1902-Z-7") (footprint "AH1902Z7")
+      (reference "IC2") (unit 1) (value "AH1902-Z-7") (footprint "HallSensor:AH1902Z7")
     )
     (path "/a6b1e09a-8af3-4cc4-9df1-f67a0e8f20fc/94b7b858-992d-497a-bd6b-051f4dea2255"
-      (reference "IC3") (unit 1) (value "AH1902-Z-7") (footprint "AH1902Z7")
+      (reference "IC3") (unit 1) (value "AH1902-Z-7") (footprint "HallSensor:AH1902Z7")
     )
     (path "/a6b1e09a-8af3-4cc4-9df1-f67a0e8f20fc/7b3f904b-56d8-43af-af24-37ea6851b116"
-      (reference "IC4") (unit 1) (value "AH1902-Z-7") (footprint "AH1902Z7")
+      (reference "IC4") (unit 1) (value "AH1902-Z-7") (footprint "HallSensor:AH1902Z7")
     )
     (path "/4afba3fc-9c59-47b9-9f58-f71bedabd29c"

Commit message: Big coils
Connections:
- net GND: now also J1.4 (Pin_4), J2.4 (Pin_4), U1.1 (EP), U1.2 (EP), U1.3 (EP), U1.4 (EP)
- net NSEROutput: now also J1.3 (Pin_3); no longer J1.4 (Pin_4)
- net VBus: now also J1.2 (Pin_2), J2.3 (Pin_3)
Changed lines of the file:
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@@
   (junction (at 87.376 137.922) (diameter 0) (color 0 0 0 0)
   )
+  (junction (at 60.452 153.416) (diameter 0) (color 0 0 0 0)
+  )
   (junction (at 40.64 127.762) (diameter 0) (color 0 0 0 0)
   )
@@
   (junction (at 40.64 125.222) (diameter 0) (color 0 0 0 0)
   )
+  (junction (at 65.532 153.416) (diameter 0) (color 0 0 0 0)
+  )
   (junction (at 40.64 132.842) (diameter 0) (color 0 0 0 0)
   )
+  (junction (at 62.992 153.416) (diameter 0) (color 0 0 0 0)
+  )
   (junction (at 40.64 137.922) (diameter 0) (color 0 0 0 0)
   )
+  (junction (at 68.072 153.416) (diameter 0) (color 0 0 0 0)
+  )
   (wire (pts (xy 48.26 150.114) (xy 96.266 150.114))
     (stroke (width 0) (type default) (color 0 0 0 0))
@@
     (stroke (width 0) (type default) (color 0 0 0 0))
   )
+  (wire (pts (xy 65.532 146.812) (xy 65.532 153.416))
+    (stroke (width 0) (type default) (color 0 0 0 0))
+  )
   (wire (pts (xy 87.376 153.416) (xy 87.376 153.67))
     (stroke (width 0) (type default) (color 0 0 0 0))
@@
     (stroke (width 0) (type default) (color 0 0 0 0))
   )
-  (wire (pts (xy 40.64 153.416) (xy 87.376 153.416))
+  (wire (pts (xy 40.64 153.416) (xy 60.452 153.416))
+    (stroke (width 0) (type default) (color 0 0 0 0))
+  )
+  (wire (pts (xy 60.452 146.812) (xy 60.452 153.416))
     (stroke (width 0) (type default) (color 0 0 0 0))
   )
@@
     (stroke (width 0) (type default) (color 0 0 0 0))
   )
+  (wire (pts (xy 62.992 153.416) (xy 65.532 153.416))
+    (stroke (width 0) (type default) (color 0 0 0 0))
+  )
+  (wire (pts (xy 68.072 153.416) (xy 87.376 153.416))
+    (stroke (width 0) (type default) (color 0 0 0 0))
+  )
   (wire (pts (xy 74.422 132.842) (xy 87.376 132.842))
     (stroke (width 0) (type default) (color 0 0 0 0))
@@
     (stroke (width 0) (type default) (color 0 0 0 0))
   )
+  (wire (pts (xy 68.072 146.812) (xy 68.072 153.416))
+    (stroke (width 0) (type default) (color 0 0 0 0))
+  )
   (wire (pts (xy 87.376 137.922) (xy 87.376 153.416))
     (stroke (width 0) (type default) (color 0 0 0 0))
   )
+  (wire (pts (xy 62.992 146.812) (xy 62.992 153.416))
+    (stroke (width 0) (type default) (color 0 0 0 0))
+  )
   (wire (pts (xy 156.21 78.74) (xy 159.004 78.74))
     (stroke (width 0) (type default) (color 0 0 0 0))
   )
+  (wire (pts (xy 65.532 153.416) (xy 68.072 153.416))
+    (stroke (width 0) (type default) (color 0 0 0 0))
+  )
   (wire (pts (xy 87.376 132.842) (xy 87.376 137.922))
     (stroke (width 0) (type default) (color 0 0 0 0))
@@
     (stroke (width 0) (type default) (color 0 0 0 0))
   )
+  (wire (pts (xy 60.452 153.416) (xy 62.992 153.416))
+    (stroke (width 0) (type default) (color 0 0 0 0))
+  )
   (wire (pts (xy 87.376 127.762) (xy 87.376 130.302))
     (stroke (width 0) (type default) (color 0 0 0 0))
@@
     (effects (font (size 1.27 1.27)) (justify left bottom))
   )
+  (label "VBus" (at 146.812 124.714 180)
+    (effects (font (size 1.27 1.27)) (justify right bottom))
+  )
   (label "QH'" (at 113.792 88.9 0)
     (effects (font (size 1.27 1.27)) (justify left bottom))
@@
     (effects (font (size 1.27 1.27)) (justify right bottom))
   )
+  (label "NSEROutput" (at 146.812 127.254 180)
+    (effects (font (size 1.27 1.27)) (justify right bottom))
+  )
+  (label "VBus" (at 147.066 147.066 180)
+    (effects (font (size 1.27 1.27)) (justify right bottom))
+  )
   (label "Data Serial" (at 113.792 73.406 0)
     (effects (font (size 1.27 1.27)) (justify left bottom))
-  )
-  (label "NSEROutput" (at 146.812 129.794 180)
-    (effects (font (size 1.27 1.27)) (justify right bottom))
   )
   (label "ClkIn" (at 159.512 122.174 0)
@@
     (pin "B9")
   )
+  (symbol (lib_id "power:GND") (at 147.066 149.606 0) (unit 1)
+    (in_bom yes) (on_board yes) (fields_autoplaced)
+    (property "Reference" "#PWR?" (id 0) (at 147.066 155.956 0)
+      (effects (font (size 1.27 1.27)) hide)
+    )
+    (property "Value" "GND" (id 1) (at 147.066 154.94 0))
+    (property "Footprint" "" (id 2) (at 147.066 149.606 0)
+      (effects (font (size 1.27 1.27)) hide)
+    )
+    (property "Datasheet" "" (id 3) (at 147.066 149.606 0)
+      (effects (font (size 1.27 1.27)) hide)
+    )
+    (pin "1")
+  )
   (symbol (lib_id "Connector_Generic:Conn_02x04_Top_Bottom") (at 152.146 144.526 0) (unit 1)
     (in_bom yes) (on_board yes) (fields_autoplaced)
@@
     (pin "8")
   )
+  (symbol (lib_id "power:GND") (at 146.812 129.794 0) (unit 1)
+    (in_bom yes) (on_board yes) (fields_autoplaced)
+    (property "Reference" "#PWR?" (id 0) (at 146.812 136.144 0)
+      (effects (font (size 1.27 1.27)) hide)
+    )
+    (property "Value" "GND" (id 1) (at 146.812 135.128 0))
+    (property "Footprint" "" (id 2) (at 146.812 129.794 0)
+      (effects (font (size 1.27 1.27)) hide)
+    )
+    (property "Datasheet" "" (id 3) (at 146.812 129.794 0)
+      (effects (font (size 1.27 1.27)) hide)
+    )
+    (pin "1")
+  )
   (sheet (at 80.01 63.246) (size 30.988 32.258) (fields_autoplaced)
     (stroke (width 0.1524) (type solid) (color 0 0 0 0))
@@
       (reference "#PWR013") (unit 1) (value "GND") (footprint "")
     )
+    (path "/6136ad65-ee71-4c73-8837-6b6089860a08"
+      (reference "#PWR?") (unit 1) (value "GND") (footprint "")
+    )
+    (path "/acdf798d-1afa-4215-a53d-19ed72d39c03"
+      (reference "#PWR?") (unit 1) (value "GND") (footprint "")
+    )
     (path "/a6b1e09a-8af3-4cc4-9df1-f67a0e8f20fc/283de13d-7f80-4c60-ab8c-dabe2f24e9cc"

Commit message: Big saucy business
Parts:
- added J3: Conn_02x04_Top_Bottom, Connector_PinHeader_2.54mm:PinHeader_2x04_P2.54mm_Vertical_SMD, symbol Connector_Generic:Conn_02x04_Top_Bottom
Connections:
- net GND: now also J3.4 (Pin_4)
- net VBus: now also J3.1 (Pin_1); no longer J1.2 (Pin_2)
- new net 5V: J1.2 (Pin_2)
Other:
- sheet Coils ports: added Vbus; removed none
Changed lines of the file:
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@@
+    (stroke (width 0) (type default) (color 0 0 0 0))
+  )
+  (wire (pts (xy 110.998 67.31) (xy 113.792 67.31))
     (stroke (width 0) (type default) (color 0 0 0 0))
   )
@@
     (effects (font (size 1.27 1.27)) (justify left bottom))
   )
-  (label "VBus" (at 146.812 124.714 180)
+  (label "VBus" (at 180.594 120.65 180)
     (effects (font (size 1.27 1.27)) (justify right bottom))
   )
@@
     (effects (font (size 1.27 1.27)) (justify left bottom))
   )
-  (label "VBus" (at 113.792 70.358 0)
+  (label "VBus" (at 113.792 67.31 0)
     (effects (font (size 1.27 1.27)) (justify left bottom))
   )
@@
     (effects (font (size 1.27 1.27)) (justify left bottom))
   )
+  (label "5V" (at 146.812 124.714 180)
+    (effects (font (size 1.27 1.27)) (justify right bottom))
+  )
   (label "NPL" (at 156.21 81.788 180)
     (effects (font (size 1.27 1.27)) (justify right bottom))
@@
     (effects (font (size 1.27 1.27)) (justify left bottom))
   )
+  (label "5V" (at 113.792 70.358 0)
+    (effects (font (size 1.27 1.27)) (justify left bottom))
+  )
   (label "NMR" (at 113.792 86.106 0)
     (effects (font (size 1.27 1.27)) (justify left bottom))
   )
-  (label "VBus" (at 156.21 68.58 180)
+  (label "5V" (at 156.21 68.58 180)
     (effects (font (size 1.27 1.27)) (justify right bottom))
   )
@@
     (pin "1")
     (pin "2")
+  )
+  (symbol (lib_id "power:GND") (at 180.594 128.27 0) (unit 1)
+    (in_bom yes) (on_board yes) (fields_autoplaced)
+    (property "Reference" "#PWR04" (id 0) (at 180.594 134.62 0)
+      (effects (font (size 1.27 1.27)) hide)
+    )
+    (property "Value" "GND" (id 1) (at 180.594 133.604 0))
+    (property "Footprint" "" (id 2) (at 180.594 128.27 0)
+      (effects (font (size 1.27 1.27)) hide)
+    )
+    (property "Datasheet" "" (id 3) (at 180.594 128.27 0)
+      (effects (font (size 1.27 1.27)) hide)
+    )
+    (pin "1")
   )
   (symbol (lib_id "power:GND") (at 87.376 153.67 0) (unit 1)
@@
   (symbol (lib_id "power:GND") (at 147.066 149.606 0) (unit 1)
     (in_bom yes) (on_board yes) (fields_autoplaced)
-    (property "Reference" "#PWR0101" (id 0) (at 147.066 155.956 0)
+    (property "Reference" "#PWR03" (id 0) (at 147.066 155.956 0)
       (effects (font (size 1.27 1.27)) hide)
     )
@@
   (symbol (lib_id "power:GND") (at 146.812 129.794 0) (unit 1)
     (in_bom yes) (on_board yes) (fields_autoplaced)
-    (property "Reference" "#PWR0102" (id 0) (at 146.812 136.144 0)
+    (property "Reference" "#PWR02" (id 0) (at 146.812 136.144 0)
       (effects (font (size 1.27 1.27)) hide)
     )
@@
     )
     (pin "1")
+  )
+  (symbol (lib_id "Connector_Generic:Conn_02x04_Top_Bottom") (at 185.674 123.19 0) (unit 1)
+    (in_bom yes) (on_board yes) (fields_autoplaced)
+    (property "Reference" "J3" (id 0) (at 186.944 114.046 0))
+    (property "Value" "Conn_02x04_Top_Bottom" (id 1) (at 186.944 116.586 0))
+    (property "Footprint" "Connector_PinHeader_2.54mm:PinHeader_2x04_P2.54mm_Vertical_SMD" (id 2) (at 185.674 123.19 0)
+      (effects (font (size 1.27 1.27)) hide)
+    )
+    (property "Datasheet" "~" (id 3) (at 185.674 123.19 0)
+      (effects (font (size 1.27 1.27)) hide)
+    )
+    (pin "1")
+    (pin "2")
+    (pin "3")
+    (pin "4")
+    (pin "5")
+    (pin "6")
+    (pin "7")
+    (pin "8")
   )
   (sheet (at 80.01 63.246) (size 30.988 32.258) (fields_autoplaced)
@@
       (effects (font (size 1.27 1.27)) (justify right))
     )
+    (pin "Vbus" input (at 110.998 67.31 0)
+      (effects (font (size 1.27 1.27)) (justify right))
+    )
   )
   (sheet (at 159.004 63.5) (size 29.464 33.02) (fields_autoplaced)
@@
       (reference "#PWR01") (unit 1) (value "GND") (footprint "")
     )
+    (path "/acdf798d-1afa-4215-a53d-19ed72d39c03"
+      (reference "#PWR02") (unit 1) (value "GND") (footprint "")
+    )
+    (path "/6136ad65-ee71-4c73-8837-6b6089860a08"
+      (reference "#PWR03") (unit 1) (value "GND") (footprint "")
+    )
+    (path "/28217338-5bf7-4267-bbae-9f97281ae53d"
+      (reference "#PWR04") (unit 1) (value "GND") (footprint "")
+    )
     (path "/590c1e64-bea6-4659-9fa3-7b726d55c0d8/cdb9a0e2-cf2e-4003-b5c9-8bddb9e96904"
-      (reference "#PWR02") (unit 1) (value "GND") (footprint "")
+      (reference "#PWR05") (unit 1) (value "GND") (footprint "")
     )
     (path "/590c1e64-bea6-4659-9fa3-7b726d55c0d8/8ef5c30c-bae0-4477-83a0-f523306a6b4f"
-      (reference "#PWR03") (unit 1) (value "GND") (footprint "")
+      (reference "#PWR06") (unit 1) (value "GND") (footprint "")
     )
     (path "/590c1e64-bea6-4659-9fa3-7b726d55c0d8/4c164dbe-0d45-4160-a820-a068598fb6f1"
-      (reference "#PWR04") (unit 1) (value "GND") (footprint "")
+      (reference "#PWR07") (unit 1) (value "GND") (footprint "")
     )
     (path "/590c1e64-bea6-4659-9fa3-7b726d55c0d8/f57e3ea1-968e-437f-a01c-e7f58eb68f1e"
-      (reference "#PWR05") (unit 1) (value "GND") (footprint "")
+      (reference "#PWR08") (unit 1) (value "GND") (footprint "")
     )
     (path "/590c1e64-bea6-4659-9fa3-7b726d55c0d8/63c334ea-ad4d-4a6e-a106-ab71c238cf05"
-      (reference "#PWR06") (unit 1) (value "GND") (footprint "")
+      (reference "#PWR09") (unit 1) (value "GND") (footprint "")
     )
     (path "/a6b1e09a-8af3-4cc4-9df1-f67a0e8f20fc/2cd2ccc8-7213-423e-8bb8-00853dfbf75d"
-      (reference "#PWR07") (unit 1) (value "GND") (footprint "")
+      (reference "#PWR010") (unit 1) (value "GND") (footprint "")
     )
     (path "/a6b1e09a-8af3-4cc4-9df1-f67a0e8f20fc/108a5baa-88b9-4907-90c0-71f684ce68bf"
-      (reference "#PWR08") (unit 1) (value "GND") (footprint "")
+      (reference "#PWR011") (unit 1) (value "GND") (footprint "")
     )
     (path "/a6b1e09a-8af3-4cc4-9df1-f67a0e8f20fc/e2ae4db1-2e25-496a-9525-9be1ecf12c6d"
-      (reference "#PWR09") (unit 1) (value "GND") (footprint "")
+      (reference "#PWR012") (unit 1) (value "GND") (footprint "")
     )
     (path "/a6b1e09a-8af3-4cc4-9df1-f67a0e8f20fc/b3a211ab-cde8-4082-b259-f7f4a4cc663f"
-      (reference "#PWR010") (unit 1) (value "GND") (footprint "")
+      (reference "#PWR013") (unit 1) (value "GND") (footprint "")
     )
     (path "/a6b1e09a-8af3-4cc4-9df1-f67a0e8f20fc/90bfdf0e-1491-4904-8db8-cf5e40170b4e"
-      (reference "#PWR011") (unit 1) (value "GND") (footprint "")
+      (reference "#PWR014") (unit 1) (value "GND") (footprint "")
     )
     (path "/a6b1e09a-8af3-4cc4-9df1-f67a0e8f20fc/fcf7c376-905e-4f32-a487-bc8568d498bd"
-      (reference "#PWR012") (unit 1) (value "GND") (footprint "")
+      (reference "#PWR015") (unit 1) (value "GND") (footprint "")
     )
     (path "/a6b1e09a-8af3-4cc4-9df1-f67a0e8f20fc/c873ee13-bc72-41e5-a1ae-57ece8d4a9f5"
-      (reference "#PWR013") (unit 1) (value "GND") (footprint "")
-    )
-    (path "/6136ad65-ee71-4c73-8837-6b6089860a08"
-      (reference "#PWR0101") (unit 1) (value "GND") (footprint "")
-    )
-    (path "/acdf798d-1afa-4215-a53d-19ed72d39c03"
-      (reference "#PWR0102") (unit 1) (value "GND") (footprint "")
+      (reference "#PWR016") (unit 1) (value "GND") (footprint "")
+    )
+    (path "/590c1e64-bea6-4659-9fa3-7b726d55c0d8/bdda89af-c175-4816-82d3-d595653a346e"
+      (reference "C1") (unit 1) (value "10u") (footprint "Capacitor_SMD:C_0805_2012Metric")
+    )
+    (path "/a6b1e09a-8af3-4cc4-9df1-f67a0e8f20fc/83dbc313-508f-4448-b6de-5809a267b5a6"
+      (reference "C2") (unit 1) (value "10u") (footprint "Capacitor_SMD:C_0805_2012Metric")
     )
     (path "/a6b1e09a-8af3-4cc4-9df1-f67a0e8f20fc/283de13d-7f80-4c60-ab8c-dabe2f24e9cc"
-      (reference "C1") (unit 1) (value "0.1u") (footprint "Capacitor_SMD:C_0402_1005Metric")
+      (reference "C3") (unit 1) (value "0.1u") (footprint "Capacitor_SMD:C_0402_1005Metric")
     )
     (path "/a6b1e09a-8af3-4cc4-9df1-f67a0e8f20fc/c8d4a300-c721-4e8e-8421-e824840dd3a3"
-      (reference "C2") (unit 1) (value "0.1u") (footprint "Capacitor_SMD:C_0402_1005Metric")
+      (reference "C4") (unit 1) (value "0.1u") (footprint "Capacitor_SMD:C_0402_1005Metric")
     )
     (path "/a6b1e09a-8af3-4cc4-9df1-f67a0e8f20fc/2f12269c-604b-4f0c-b6d2-570b375e6f3e"
-      (reference "C3") (unit 1) (value "0.1u") (footprint "Capacitor_SMD:C_0402_1005Metric")
+      (reference "C5") (unit 1) (value "0.1u") (footprint "Capacitor_SMD:C_0402_1005Metric")
     )
     (path "/a6b1e09a-8af3-4cc4-9df1-f67a0e8f20fc/004e570a-651a-4298-8191-ceec66973458"
-      (reference "C4") (unit 1) (value "0.1u") (footprint "Capacitor_SMD:C_0402_1005Metric")
+      (reference "C6") (unit 1) (value "0.1u") (footprint "Capacitor_SMD:C_0402_1005Metric")
     )
     (path "/06df2c7b-9992-4fe2-8804-c49a5197fa1a"
@@
       (reference "J2") (unit 1) (value "Conn_02x04_Top_Bottom") (footprint "Connector_PinHeader_2.54mm:PinHeader_2x04_P2.54mm_Vertical_SMD")
     )
+    (path "/f3245e87-e57c-4a07-8e6c-7d6293b755be"
+      (reference "J3") (unit 1) (value "Conn_02x04_Top_Bottom") (footprint "Connector_PinHeader_2.54mm:PinHeader_2x04_P2.54mm_Vertical_SMD")
+    )
     (path "/590c1e64-bea6-4659-9fa3-7b726d55c0d8/70f43254-c71c-407a-929e-cc599b9c2a26"
