File: KiCad Files/RowdyTestBoard2.kicad_sch (KiCad schematic)
At the start: 5 parts, among them J1 Conn_02x04_Top_Bottom, J2 Conn_02x04_Top_Bottom, J3 Conn_02x04_Top_Bottom, U1 USB-C

Commit message: Big coils baby
Parts:
- removed D1: 1N5819, Diode_SMD:D_SOD-323F, symbol Diode:1N5819
- removed U1: USB-C, USB_C:USB-C-SMD_KH-TYPE-C-16P, symbol usb-c:USB-C
Connections:
- net VBus renamed Vcc

Commit message: Final pt 1
Other:
- company: (none) -> Rowdy Chess
- title: (none) -> Rowdy Test Board
Changed lines of the file:
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@@
 (kicad_sch (version 20211123) (generator eeschema)
   (paper "A4")
+  (title_block
+    (title "Rowdy Test Board")
+    (date "2022-06-26")
+    (company "Rowdy Chess")
+    (comment 1 "Authors: Daniel Jones, David Newton, Mishay Naidoo")
+  )
   (wire (pts (xy 110.998 79.756) (xy 113.792 79.756))
     (stroke (width 0) (type default) (color 0 0 0 0))

Commit message: Generated JLC PCB Files
Parts:
- J1, J2, J3: JLC Part Number (none) -> C192300; LCSC (none) -> C192300
Changed lines of the file:
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@@
+      (effects (font (size 1.27 1.27)) hide)
+    )
+    (property "JLC Part Number" "C192300" (id 4) (at 151.892 124.714 0)
+      (effects (font (size 1.27 1.27)) hide)
+    )
+    (property "LCSC" "C192300" (id 5) (at 151.892 124.714 0)
       (effects (font (size 1.27 1.27)) hide)
     )
@@
       (effects (font (size 1.27 1.27)) hide)
     )
+    (property "JLC Part Number" "C192300" (id 4) (at 152.146 144.526 0)
+      (effects (font (size 1.27 1.27)) hide)
+    )
+    (property "LCSC" "C192300" (id 5) (at 152.146 144.526 0)
+      (effects (font (size 1.27 1.27)) hide)
+    )
     (pin "1")
     (pin "2")
@@
       (effects (font (size 1.27 1.27)) hide)
     )
+    (property "JLC Part Number" "C192300" (id 4) (at 185.674 123.19 0)
+      (effects (font (size 1.27 1.27)) hide)
+    )
+    (property "LCSC" "C192300" (id 5) (at 185.674 123.19 0)
+      (effects (font (size 1.27 1.27)) hide)
+    )
