File: KiCad Files/power.kicad_sch (KiCad schematic)
At the start: 0 parts

Commit message: More footprints
Parts:
- added U3: USB-C, USB_C:USB-C-SMD_KH-TYPE-C-16P, symbol usb-c:USB-C
Changed lines of the file:
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@@
 (kicad_sch (version 20211123) (generator eeschema)
   (paper "A4")
+  (symbol (lib_id "usb-c:USB-C") (at 96.52 53.34 0) (unit 1)
+    (in_bom yes) (on_board yes) (fields_autoplaced)
+    (property "Reference" "U3" (id 0) (at 96.52 34.29 0))
+    (property "Value" "USB-C" (id 1) (at 96.52 36.83 0))
+    (property "Footprint" "USB_C:USB-C-SMD_KH-TYPE-C-16P" (id 2) (at 96.52 53.34 0)
+      (effects (font (size 1.27 1.27)) hide)
+    )
+    (property "Datasheet" "https://datasheet.lcsc.com/lcsc/2009111434_Shenzhen-Kinghelm-Elec-KH-TYPE-C-16P_C709357.pdf" (id 3) (at 96.52 53.34 0)
+      (effects (font (size 1.27 1.27)) hide)
+    )
+    (property "JLC Part Number" "C709357" (id 4) (at 96.52 53.34 0)
+      (effects (font (size 1.27 1.27)) hide)
+    )
+    (pin "1")
+    (pin "2")
+    (pin "3")
+    (pin "4")
+    (pin "A1")
+    (pin "A12")
+    (pin "A4")
+    (pin "A5")
+    (pin "A6")
+    (pin "A7")
+    (pin "A8")
+    (pin "A9")
+    (pin "B1")
+    (pin "B12")
+    (pin "B4")
+    (pin "B5")
+    (pin "B6")
+    (pin "B7")
+    (pin "B8")
+    (pin "B9")
+  )
 )

Commit message: Pcb2
Connections:
- net GND: now reaches U3.A1 (GND)
- net GND: now also U3.A12 (GND), U3.A5 (CC1), U3.A6 (DP1), U3.A7 (DN1), U3.A8 (SUB1), U3.B1 (GND), U3.B12 (GND), U3.B5 (CC2), U3.B6 (DP2), U3.B7 (DN2), U3.B8 (SUB2)
- net VBUS: now reaches U3.A4 (VBUS)
- net VBUS: now also U3.A9 (VBUS), U3.B4 (VBUS), U3.B9 (VBUS)
Other:
- moved on the sheet: U3
Changed lines of the file:
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@@
 (kicad_sch (version 20211123) (generator eeschema)
   (paper "A4")
-  (symbol (lib_id "usb-c:USB-C") (at 96.52 53.34 0) (unit 1)
+  (junction (at 118.872 77.978) (diameter 0) (color 0 0 0 0)
+  )
+  (junction (at 118.872 72.898) (diameter 0) (color 0 0 0 0)
+  )
+  (junction (at 118.872 75.438) (diameter 0) (color 0 0 0 0)
+  )
+  (junction (at 72.136 70.358) (diameter 0) (color 0 0 0 0)
+  )
+  (junction (at 118.872 98.552) (diameter 0) (color 0 0 0 0)
+  )
+  (junction (at 72.136 83.058) (diameter 0) (color 0 0 0 0)
+  )
+  (junction (at 72.136 75.438) (diameter 0) (color 0 0 0 0)
+  )
+  (junction (at 127.762 80.518) (diameter 0) (color 0 0 0 0)
+  )
+  (junction (at 127.762 67.818) (diameter 0) (color 0 0 0 0)
+  )
+  (junction (at 118.872 83.058) (diameter 0) (color 0 0 0 0)
+  )
+  (junction (at 72.136 72.898) (diameter 0) (color 0 0 0 0)
+  )
+  (junction (at 118.872 70.358) (diameter 0) (color 0 0 0 0)
+  )
+  (junction (at 72.136 77.978) (diameter 0) (color 0 0 0 0)
+  )
+  (wire (pts (xy 85.598 80.518) (xy 79.756 80.518))
+    (stroke (width 0) (type default) (color 0 0 0 0))
+  )
+  (wire (pts (xy 118.872 75.438) (xy 118.872 77.978))
+    (stroke (width 0) (type default) (color 0 0 0 0))
+  )
+  (wire (pts (xy 72.136 98.552) (xy 118.872 98.552))
+    (stroke (width 0) (type default) (color 0 0 0 0))
+  )
+  (wire (pts (xy 85.598 67.818) (xy 79.756 67.818))
+    (stroke (width 0) (type default) (color 0 0 0 0))
+  )
+  (wire (pts (xy 127.762 67.818) (xy 135.89 67.818))
+    (stroke (width 0) (type default) (color 0 0 0 0))
+  )
+  (wire (pts (xy 118.872 83.058) (xy 118.872 98.552))
+    (stroke (width 0) (type default) (color 0 0 0 0))
+  )
+  (wire (pts (xy 105.918 67.818) (xy 127.762 67.818))
+    (stroke (width 0) (type default) (color 0 0 0 0))
+  )
+  (wire (pts (xy 79.756 80.518) (xy 79.756 95.25))
+    (stroke (width 0) (type default) (color 0 0 0 0))
+  )
+  (wire (pts (xy 72.136 75.438) (xy 85.598 75.438))
+    (stroke (width 0) (type default) (color 0 0 0 0))
+  )
+  (wire (pts (xy 72.136 65.278) (xy 72.136 70.358))
+    (stroke (width 0) (type default) (color 0 0 0 0))
+  )
+  (wire (pts (xy 118.872 77.978) (xy 118.872 83.058))
+    (stroke (width 0) (type default) (color 0 0 0 0))
+  )
+  (wire (pts (xy 72.136 83.058) (xy 72.136 98.552))
+    (stroke (width 0) (type default) (color 0 0 0 0))
+  )
+  (wire (pts (xy 72.136 70.358) (xy 85.598 70.358))
+    (stroke (width 0) (type default) (color 0 0 0 0))
+  )
+  (wire (pts (xy 72.136 70.358) (xy 72.136 72.898))
+    (stroke (width 0) (type default) (color 0 0 0 0))
+  )
+  (wire (pts (xy 79.756 95.25) (xy 127.762 95.25))
+    (stroke (width 0) (type default) (color 0 0 0 0))
+  )
+  (wire (pts (xy 105.918 83.058) (xy 118.872 83.058))
+    (stroke (width 0) (type default) (color 0 0 0 0))
+  )
+  (wire (pts (xy 135.89 67.818) (xy 135.89 55.372))
+    (stroke (width 0) (type default) (color 0 0 0 0))
+  )
+  (wire (pts (xy 118.872 98.552) (xy 118.872 98.806))
+    (stroke (width 0) (type default) (color 0 0 0 0))
+  )
+  (wire (pts (xy 85.598 65.278) (xy 72.136 65.278))
+    (stroke (width 0) (type default) (color 0 0 0 0))
+  )
+  (wire (pts (xy 72.136 83.058) (xy 85.598 83.058))
+    (stroke (width 0) (type default) (color 0 0 0 0))
+  )
+  (wire (pts (xy 127.762 80.518) (xy 127.762 67.818))
+    (stroke (width 0) (type default) (color 0 0 0 0))
+  )
+  (wire (pts (xy 105.918 75.438) (xy 118.872 75.438))
+    (stroke (width 0) (type default) (color 0 0 0 0))
+  )
+  (wire (pts (xy 105.918 80.518) (xy 127.762 80.518))
+    (stroke (width 0) (type default) (color 0 0 0 0))
+  )
+  (wire (pts (xy 79.756 54.102) (xy 127.762 54.102))
+    (stroke (width 0) (type default) (color 0 0 0 0))
+  )
+  (wire (pts (xy 127.762 54.102) (xy 127.762 67.818))
+    (stroke (width 0) (type default) (color 0 0 0 0))
+  )
+  (wire (pts (xy 118.872 65.278) (xy 118.872 70.358))
+    (stroke (width 0) (type default) (color 0 0 0 0))
+  )
+  (wire (pts (xy 72.136 77.978) (xy 85.598 77.978))
+    (stroke (width 0) (type default) (color 0 0 0 0))
+  )
+  (wire (pts (xy 105.918 72.898) (xy 118.872 72.898))
+    (stroke (width 0) (type default) (color 0 0 0 0))
+  )
+  (wire (pts (xy 72.136 72.898) (xy 72.136 75.438))
+    (stroke (width 0) (type default) (color 0 0 0 0))
+  )
+  (wire (pts (xy 118.872 70.358) (xy 118.872 72.898))
+    (stroke (width 0) (type default) (color 0 0 0 0))
+  )
+  (wire (pts (xy 105.918 70.358) (xy 118.872 70.358))
+    (stroke (width 0) (type default) (color 0 0 0 0))
+  )
+  (wire (pts (xy 72.136 75.438) (xy 72.136 77.978))
+    (stroke (width 0) (type default) (color 0 0 0 0))
+  )
+  (wire (pts (xy 72.136 72.898) (xy 85.598 72.898))
+    (stroke (width 0) (type default) (color 0 0 0 0))
+  )
+  (wire (pts (xy 72.136 77.978) (xy 72.136 83.058))
+    (stroke (width 0) (type default) (color 0 0 0 0))
+  )
+  (wire (pts (xy 79.756 67.818) (xy 79.756 54.102))
+    (stroke (width 0) (type default) (color 0 0 0 0))
+  )
+  (wire (pts (xy 118.872 72.898) (xy 118.872 75.438))
+    (stroke (width 0) (type default) (color 0 0 0 0))
+  )
+  (wire (pts (xy 105.918 77.978) (xy 118.872 77.978))
+    (stroke (width 0) (type default) (color 0 0 0 0))
+  )
+  (wire (pts (xy 127.762 95.25) (xy 127.762 80.518))
+    (stroke (width 0) (type default) (color 0 0 0 0))
+  )
+  (wire (pts (xy 105.918 65.278) (xy 118.872 65.278))
+    (stroke (width 0) (type default) (color 0 0 0 0))
+  )
+  (hierarchical_label "VBUS" (shape input) (at 135.89 55.372 0)
+    (effects (font (size 1.27 1.27)) (justify left))
+  )
+  (symbol (lib_id "usb-c:USB-C") (at 95.758 75.438 0) (unit 1)
     (in_bom yes) (on_board yes) (fields_autoplaced)
-    (property "Reference" "U3" (id 0) (at 96.52 34.29 0))
-    (property "Value" "USB-C" (id 1) (at 96.52 36.83 0))
-    (property "Footprint" "USB_C:USB-C-SMD_KH-TYPE-C-16P" (id 2) (at 96.52 53.34 0)
+    (property "Reference" "U3" (id 0) (at 95.758 56.388 0))
+    (property "Value" "USB-C" (id 1) (at 95.758 58.928 0))
+    (property "Footprint" "USB_C:USB-C-SMD_KH-TYPE-C-16P" (id 2) (at 95.758 75.438 0)
       (effects (font (size 1.27 1.27)) hide)
     )
-    (property "Datasheet" "https://datasheet.lcsc.com/lcsc/2009111434_Shenzhen-Kinghelm-Elec-KH-TYPE-C-16P_C709357.pdf" (id 3) (at 96.52 53.34 0)
+    (property "Datasheet" "https://datasheet.lcsc.com/lcsc/2009111434_Shenzhen-Kinghelm-Elec-KH-TYPE-C-16P_C709357.pdf" (id 3) (at 95.758 75.438 0)
       (effects (font (size 1.27 1.27)) hide)
     )
-    (property "JLC Part Number" "C709357" (id 4) (at 96.52 53.34 0)
+    (property "JLC Part Number" "C709357" (id 4) (at 95.758 75.438 0)
       (effects (font (size 1.27 1.27)) hide)
     )
@@
     (pin "B9")
   )
+  (symbol (lib_id "power:GND") (at 118.872 98.806 0) (unit 1)
+    (in_bom yes) (on_board yes) (fields_autoplaced)
+    (property "Reference" "#PWR?" (id 0) (at 118.872 105.156 0)
+      (effects (font (size 1.27 1.27)) hide)
+    )
+    (property "Value" "GND" (id 1) (at 118.872 104.14 0))
+    (property "Footprint" "" (id 2) (at 118.872 98.806 0)
+      (effects (font (size 1.27 1.27)) hide)
+    )
+    (property "Datasheet" "" (id 3) (at 118.872 98.806 0)
+      (effects (font (size 1.27 1.27)) hide)
+    )
+    (pin "1")
+  )
 )
