File: KiCad Files/RowdyTestBoard2.kicad_pcb (KiCad board)
At the start: 4 copper layers, 0 parts

Commit message: Pcb2
Parts:
- added C1: 0.1u, Capacitor_SMD:C_0402_1005Metric, F.Cu at (144.3, 80.5)
- added C2: 0.1u, Capacitor_SMD:C_0402_1005Metric, F.Cu at (144.3, 82.5)
- added C3: 0.1u, Capacitor_SMD:C_0402_1005Metric, F.Cu at (147.1, 78.5)
- added C4: 0.1u, Capacitor_SMD:C_0402_1005Metric, F.Cu at (144.3, 78.5)
- added D1: 1N5819, Diode_THT:D_DO-41_SOD81_P10.16mm_Horizontal, F.Cu at (161.5, 84.7)
- added J1: Conn_02x04_Top_Bottom, Connector_PinHeader_2.54mm:PinHeader_2x04_P2.54mm_Vertical_SMD, F.Cu at (117.9, 67.2)
- added J2: Conn_02x04_Top_Bottom, Connector_PinHeader_2.54mm:PinHeader_2x04_P2.54mm_Vertical_SMD, F.Cu at (130.7, 67.2)
- added Q1: AO3400A, Package_TO_SOT_SMD:SOT-23, F.Cu at (145.3, 72.2)
- added Q2: AO3400A, Package_TO_SOT_SMD:SOT-23, F.Cu at (150.2, 63.3)
- added Q3: AO3400A, Package_TO_SOT_SMD:SOT-23, F.Cu at (145.3, 67.7)
- added Q4: AO3400A, Package_TO_SOT_SMD:SOT-23, F.Cu at (150.2, 67.7)
- added Q5: AO3401A, Package_TO_SOT_SMD:SOT-23, F.Cu at (155.1, 63.3)
- added Q6: AO3401A, Package_TO_SOT_SMD:SOT-23, F.Cu at (145.3, 63.3)
- added Q7: AO3401A, Package_TO_SOT_SMD:SOT-23, F.Cu at (150.2, 72.2)
- added Q8: AO3401A, Package_TO_SOT_SMD:SOT-23, F.Cu at (155.1, 67.7)

Commit message: diode
Parts:
- added IC1: AH1902-Z-7, HallSensor:AH1902Z7, F.Cu at (119.9, 96.4)
- added IC2: AH1902-Z-7, HallSensor:AH1902Z7, F.Cu at (115.2, 90.4)
- added IC3: AH1902-Z-7, HallSensor:AH1902Z7, F.Cu at (119.9, 90.4)
- added IC4: AH1902-Z-7, HallSensor:AH1902Z7, F.Cu at (115.2, 96.4)
- added U1: USB-C, USB_C:USB-C-SMD_KH-TYPE-C-16P, F.Cu at (134.2, 90.7)
- added U2: 74HC595, 74HC595:SO16, F.Cu at (134.4, 103.9)
- added U3: 74HC165, 74HC165:SO-16, F.Cu at (107.3, 92.2)
