File: KiCad Files/sensors.kicad_sch (KiCad schematic)
At the start: 9 parts, among them IC1 AH1902-Z-7, IC2 AH1902-Z-7, IC3 AH1902-Z-7, IC4 AH1902-Z-7, U3 74HC165

Commit message: diode
Parts:
- IC1, IC2, IC3, IC4: footprint AH1902Z7 -> HallSensor:AH1902Z7
Changed lines of the file:
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@@
     (property "Reference" "IC2" (id 0) (at 156.718 55.626 0))
     (property "Value" "AH1902-Z-7" (id 1) (at 156.718 58.166 0))
-    (property "Footprint" "AH1902Z7" (id 2) (at 168.148 60.452 0)
+    (property "Footprint" "HallSensor:AH1902Z7" (id 2) (at 168.148 60.452 0)
       (effects (font (size 1.27 1.27)) (justify left) hide)
     )
@@
     (property "Reference" "IC4" (id 0) (at 156.718 88.138 0))
     (property "Value" "AH1902-Z-7" (id 1) (at 156.718 90.678 0))
-    (property "Footprint" "AH1902Z7" (id 2) (at 168.148 92.964 0)
+    (property "Footprint" "HallSensor:AH1902Z7" (id 2) (at 168.148 92.964 0)
       (effects (font (size 1.27 1.27)) (justify left) hide)
     )
@@
     (property "Reference" "IC3" (id 0) (at 156.718 71.882 0))
     (property "Value" "AH1902-Z-7" (id 1) (at 156.718 74.422 0))
-    (property "Footprint" "AH1902Z7" (id 2) (at 168.148 76.708 0)
+    (property "Footprint" "HallSensor:AH1902Z7" (id 2) (at 168.148 76.708 0)
       (effects (font (size 1.27 1.27)) (justify left) hide)
     )
@@
     (property "Reference" "IC1" (id 0) (at 156.718 39.37 0))
     (property "Value" "AH1902-Z-7" (id 1) (at 156.718 41.91 0))
-    (property "Footprint" "AH1902Z7" (id 2) (at 168.148 44.196 0)
-      (effects (font (size 1.27 1.27)) (justify left) hide)
-    )
+    (property "Footprint" "HallSensor:AH1902Z7" (id 2) (at 168.148 44.196 0)
+      (effects (font (size 1.27 1.27)) (justify left) hide)
+    )

Commit message: Big saucy business
Parts:
- added C2: 10u, Capacitor_SMD:C_0805_2012Metric, symbol Device:C
- renumbered C1 to C3, C2 to C4, C3 to C5, C4 to C6
Connections:
- net 5V: now also C2.1
- net GND: now also C2.2
Changed lines of the file:
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@@
   (junction (at 112.014 67.056) (diameter 0) (color 0 0 0 0)
   )
+  (junction (at 97.028 37.338) (diameter 0) (color 0 0 0 0)
+  )
   (junction (at 171.958 98.044) (diameter 0) (color 0 0 0 0)
   )
@@
   (junction (at 171.958 49.276) (diameter 0) (color 0 0 0 0)
   )
+  (junction (at 97.028 87.63) (diameter 0) (color 0 0 0 0)
+  )
   (junction (at 138.43 95.504) (diameter 0) (color 0 0 0 0)
   )
@@
     (stroke (width 0) (type default) (color 0 0 0 0))
   )
+  (wire (pts (xy 61.976 37.338) (xy 61.976 44.196))
+    (stroke (width 0) (type default) (color 0 0 0 0))
+  )
   (wire (pts (xy 112.014 46.736) (xy 112.014 59.436))
     (stroke (width 0) (type default) (color 0 0 0 0))
   )
-  (wire (pts (xy 97.028 35.814) (xy 97.028 39.116))
+  (wire (pts (xy 97.028 35.814) (xy 97.028 37.338))
     (stroke (width 0) (type default) (color 0 0 0 0))
   )
@@
     (stroke (width 0) (type default) (color 0 0 0 0))
   )
+  (wire (pts (xy 97.028 87.63) (xy 97.028 87.884))
+    (stroke (width 0) (type default) (color 0 0 0 0))
+  )
   (wire (pts (xy 171.958 68.072) (xy 171.958 71.374))
     (stroke (width 0) (type default) (color 0 0 0 0))
@@
     (stroke (width 0) (type default) (color 0 0 0 0))
   )
+  (wire (pts (xy 97.028 37.338) (xy 97.028 39.116))
+    (stroke (width 0) (type default) (color 0 0 0 0))
+  )
   (wire (pts (xy 171.958 100.584) (xy 171.958 103.886))
     (stroke (width 0) (type default) (color 0 0 0 0))
@@
     (stroke (width 0) (type default) (color 0 0 0 0))
   )
+  (wire (pts (xy 97.028 87.376) (xy 97.028 87.63))
+    (stroke (width 0) (type default) (color 0 0 0 0))
+  )
   (wire (pts (xy 137.922 59.436) (xy 134.62 59.436))
     (stroke (width 0) (type default) (color 0 0 0 0))
@@
     (stroke (width 0) (type default) (color 0 0 0 0))
   )
+  (wire (pts (xy 97.028 37.338) (xy 61.976 37.338))
+    (stroke (width 0) (type default) (color 0 0 0 0))
+  )
+  (wire (pts (xy 61.976 87.63) (xy 97.028 87.63))
+    (stroke (width 0) (type default) (color 0 0 0 0))
+  )
   (wire (pts (xy 130.556 46.736) (xy 130.556 62.992))
+    (stroke (width 0) (type default) (color 0 0 0 0))
+  )
+  (wire (pts (xy 61.976 51.816) (xy 61.976 87.63))
     (stroke (width 0) (type default) (color 0 0 0 0))
   )
@@
   (symbol (lib_id "Device:C") (at 138.43 105.156 0) (unit 1)
     (in_bom yes) (on_board yes) (fields_autoplaced)
-    (property "Reference" "C4" (id 0) (at 142.24 103.8859 0)
+    (property "Reference" "C6" (id 0) (at 142.24 103.8859 0)
       (effects (font (size 1.27 1.27)) (justify left))
     )
@@
   (symbol (lib_id "power:GND") (at 112.014 83.566 0) (unit 1)
     (in_bom yes) (on_board yes) (fields_autoplaced)
-    (property "Reference" "#PWR08" (id 0) (at 112.014 89.916 0)
+    (property "Reference" "#PWR011" (id 0) (at 112.014 89.916 0)
       (effects (font (size 1.27 1.27)) hide)
     )
@@
   (symbol (lib_id "Device:C") (at 137.922 55.626 0) (unit 1)
     (in_bom yes) (on_board yes) (fields_autoplaced)
-    (property "Reference" "C1" (id 0) (at 141.732 54.3559 0)
+    (property "Reference" "C3" (id 0) (at 141.732 54.3559 0)
       (effects (font (size 1.27 1.27)) (justify left))
     )
@@
     (pin "2")
   )
-  (symbol (lib_id "power:GND") (at 97.028 87.376 0) (unit 1)
-    (in_bom yes) (on_board yes) (fields_autoplaced)
-    (property "Reference" "#PWR07" (id 0) (at 97.028 93.726 0)
-      (effects (font (size 1.27 1.27)) hide)
-    )
-    (property "Value" "GND" (id 1) (at 97.028 91.948 0))
-    (property "Footprint" "" (id 2) (at 97.028 87.376 0)
-      (effects (font (size 1.27 1.27)) hide)
-    )
-    (property "Datasheet" "" (id 3) (at 97.028 87.376 0)
+  (symbol (lib_id "power:GND") (at 97.028 87.884 0) (unit 1)
+    (in_bom yes) (on_board yes) (fields_autoplaced)
+    (property "Reference" "#PWR010" (id 0) (at 97.028 94.234 0)
+      (effects (font (size 1.27 1.27)) hide)
+    )
+    (property "Value" "GND" (id 1) (at 97.028 92.456 0))
+    (property "Footprint" "" (id 2) (at 97.028 87.884 0)
+      (effects (font (size 1.27 1.27)) hide)
+    )
+    (property "Datasheet" "" (id 3) (at 97.028 87.884 0)
       (effects (font (size 1.27 1.27)) hide)
     )
@@
   (symbol (lib_id "Device:C") (at 137.922 87.884 0) (unit 1)
     (in_bom yes) (on_board yes) (fields_autoplaced)
-    (property "Reference" "C3" (id 0) (at 141.732 86.6139 0)
+    (property "Reference" "C5" (id 0) (at 141.732 86.6139 0)
       (effects (font (size 1.27 1.27)) (justify left))
     )
@@
     (pin "5")
   )
+  (symbol (lib_id "Device:C") (at 61.976 48.006 0) (unit 1)
+    (in_bom yes) (on_board yes) (fields_autoplaced)
+    (property "Reference" "C2" (id 0) (at 65.786 46.7359 0)
+      (effects (font (size 1.27 1.27)) (justify left))
+    )
+    (property "Value" "10u" (id 1) (at 65.786 49.2759 0)
+      (effects (font (size 1.27 1.27)) (justify left))
+    )
+    (property "Footprint" "Capacitor_SMD:C_0805_2012Metric" (id 2) (at 62.9412 51.816 0)
+      (effects (font (size 1.27 1.27)) hide)
+    )
+    (property "Datasheet" "https://datasheet.lcsc.com/lcsc/1811121310_Samsung-Electro-Mechanics-CL21A106KAYNNNE_C15850.pdf" (id 3) (at 61.976 48.006 0)
+      (effects (font (size 1.27 1.27)) hide)
+    )
+    (property "JLC Part Number" "C15850" (id 4) (at 61.976 48.006 0)
+      (effects (font (size 1.27 1.27)) hide)
+    )
+    (pin "1")
+    (pin "2")
+  )
   (symbol (lib_id "power:GND") (at 171.958 71.374 0) (unit 1)
     (in_bom yes) (on_board yes) (fields_autoplaced)
-    (property "Reference" "#PWR011" (id 0) (at 171.958 77.724 0)
+    (property "Reference" "#PWR014" (id 0) (at 171.958 77.724 0)
       (effects (font (size 1.27 1.27)) hide)
     )
@@
   (symbol (lib_id "power:GND") (at 171.958 55.118 0) (unit 1)
     (in_bom yes) (on_board yes) (fields_autoplaced)
-    (property "Reference" "#PWR010" (id 0) (at 171.958 61.468 0)
+    (property "Reference" "#PWR013" (id 0) (at 171.958 61.468 0)
       (effects (font (size 1.27 1.27)) hide)
     )
@@
   (symbol (lib_id "power:GND") (at 171.958 103.886 0) (unit 1)
     (in_bom yes) (on_board yes) (fields_autoplaced)
-    (property "Reference" "#PWR013" (id 0) (at 171.958 110.236 0)
+    (property "Reference" "#PWR016" (id 0) (at 171.958 110.236 0)
       (effects (font (size 1.27 1.27)) hide)
     )
@@
   (symbol (lib_id "Device:C") (at 137.922 71.882 0) (unit 1)
     (in_bom yes) (on_board yes) (fields_autoplaced)
-    (property "Reference" "C2" (id 0) (at 141.732 70.6119 0)
+    (property "Reference" "C4" (id 0) (at 141.732 70.6119 0)
       (effects (font (size 1.27 1.27)) (justify left))
     )
@@
   (symbol (lib_id "power:GND") (at 138.43 112.268 0) (unit 1)
     (in_bom yes) (on_board yes) (fields_autoplaced)
-    (property "Reference" "#PWR09" (id 0) (at 138.43 118.618 0)
+    (property "Reference" "#PWR012" (id 0) (at 138.43 118.618 0)
       (effects (font (size 1.27 1.27)) hide)
     )
@@
   (symbol (lib_id "power:GND") (at 171.958 87.63 0) (unit 1)
     (in_bom yes) (on_board yes) (fields_autoplaced)
-    (property "Reference" "#PWR012" (id 0) (at 171.958 93.98 0)
-      (effects (font (size 1.27 1.27)) hide)
-    )
+    (property "Reference" "#PWR015" (id 0) (at 171.958 93.98 0)
+      (effects (font (size 1.27 1.27)) hide)
+    )
