File: KiCad Files/sensors.kicad_sch (KiCad schematic)
At the start: 10 parts, among them IC1 AH1902-Z-7, IC2 AH1902-Z-7, IC3 AH1902-Z-7, IC4 AH1902-Z-7, U3 74HC165

Commit message: Final pt 1
Other:
- company: (none) -> Rowdy Chess
- title: (none) -> Rowdy Test Board
Changed lines of the file:
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@@
 (kicad_sch (version 20211123) (generator eeschema)
   (paper "A4")
+  (title_block
+    (title "Rowdy Test Board")
+    (date "2022-06-26")
+    (company "Rowdy Chess")
+    (comment 1 "Authors: Daniel Jones, David Newton, Mishay Naidoo")
+  )
   (junction (at 134.62 75.692) (diameter 0) (color 0 0 0 0)
   )

Commit message: Generated JLC PCB Files
Parts:
- C3: LCSC (none) -> C15850
- C4, C5, C6, C7: LCSC (none) -> C1525
- IC1, IC2, IC3, IC4: LCSC (none) -> C239188
- U3: LCSC (none) -> C5613
Changed lines of the file:
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@@
+      (effects (font (size 1.27 1.27)) hide)
+    )
+    (property "LCSC" "C1525" (id 5) (at 138.43 105.156 0)
       (effects (font (size 1.27 1.27)) hide)
     )
@@
     )
     (property "JLC Part Number" "C5613" (id 4) (at 97.028 61.976 0)
+      (effects (font (size 1.27 1.27)) hide)
+    )
+    (property "LCSC" "C5613" (id 5) (at 97.028 61.976 0)
       (effects (font (size 1.27 1.27)) hide)
     )
@@
       (effects (font (size 1.27 1.27)) hide)
     )
+    (property "LCSC" "C239188" (id 13) (at 141.478 62.992 0)
+      (effects (font (size 1.27 1.27)) hide)
+    )
     (pin "1")
     (pin "2")
@@
       (effects (font (size 1.27 1.27)) hide)
     )
+    (property "LCSC" "C1525" (id 5) (at 137.922 55.626 0)
+      (effects (font (size 1.27 1.27)) hide)
+    )
     (pin "1")
     (pin "2")
@@
     )
     (property "JLC Part Number" "C1525" (id 4) (at 137.922 87.884 0)
+      (effects (font (size 1.27 1.27)) hide)
+    )
+    (property "LCSC" "C1525" (id 5) (at 137.922 87.884 0)
       (effects (font (size 1.27 1.27)) hide)
     )
@@
       (effects (font (size 1.27 1.27)) hide)
     )
+    (property "LCSC" "C239188" (id 13) (at 141.478 95.504 0)
+      (effects (font (size 1.27 1.27)) hide)
+    )
     (pin "1")
     (pin "2")
@@
       (effects (font (size 1.27 1.27)) hide)
     )
+    (property "LCSC" "C15850" (id 5) (at 61.976 48.006 0)
+      (effects (font (size 1.27 1.27)) hide)
+    )
     (pin "1")
     (pin "2")
@@
       (effects (font (size 1.27 1.27)) hide)
     )
+    (property "LCSC" "C239188" (id 13) (at 141.478 79.248 0)
+      (effects (font (size 1.27 1.27)) hide)
+    )
     (pin "1")
     (pin "2")
@@
       (effects (font (size 1.27 1.27)) hide)
     )
+    (property "LCSC" "C1525" (id 5) (at 137.922 71.882 0)
+      (effects (font (size 1.27 1.27)) hide)
+    )
     (pin "1")
     (pin "2")
@@
       (effects (font (size 1.27 1.27)) hide)
     )
+    (property "LCSC" "C239188" (id 13) (at 141.478 46.736 0)
+      (effects (font (size 1.27 1.27)) hide)
+    )

Commit message: New Hall Sensors
Parts:
- removed IC1, IC2, IC3, IC4: AH1902-Z-7, HallSensor:AH1902Z7, symbol AH1902-Z-7:AH1902-Z-7
- added U4, U5, U6, U7: SOT95, SOT95:SOT95P230X110-3N, symbol Sensor_Magnetic:A1101ELHL
Connections:
- net 3V: now also U4.1 (VCC), U5.1 (VCC), U6.1 (VCC), U7.1 (VCC)
- net GND: now also U4.3 (GND), U5.3 (GND), U6.3 (GND), U7.3 (GND)
- net at U3.11 (D0): now also U5.2 (VOUT)
- net at U3.12 (D1): now also U6.2 (VOUT)
- net at U3.13 (D2): now also U4.2 (VOUT)
- net at U3.14 (D3): now also U7.2 (VOUT)
