File: KiCad Files/sensors.kicad_sch (KiCad schematic)
At the start: 10 parts, among them IC1 AH1902-Z-7, IC2 AH1902-Z-7, IC3 AH1902-Z-7, IC4 AH1902-Z-7, U3 74HC165

Commit message: Big coils baby
Parts:
- renumbered U3 to U2
Changed lines of the file:
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@@
   (symbol (lib_id "power:GND") (at 112.014 83.566 0) (unit 1)
     (in_bom yes) (on_board yes) (fields_autoplaced)
-    (property "Reference" "#PWR011" (id 0) (at 112.014 89.916 0)
+    (property "Reference" "#PWR010" (id 0) (at 112.014 89.916 0)
       (effects (font (size 1.27 1.27)) hide)
     )
@@
   (symbol (lib_id "74xx:74HC165") (at 97.028 61.976 0) (mirror y) (unit 1)
     (in_bom yes) (on_board yes) (fields_autoplaced)
-    (property "Reference" "U3" (id 0) (at 97.5486 39.116 0)
+    (property "Reference" "U2" (id 0) (at 97.5486 39.116 0)
       (effects (font (size 1.27 1.27)) (justify right))
     )
@@
   (symbol (lib_id "power:GND") (at 97.028 87.884 0) (unit 1)
     (in_bom yes) (on_board yes) (fields_autoplaced)
-    (property "Reference" "#PWR010" (id 0) (at 97.028 94.234 0)
+    (property "Reference" "#PWR09" (id 0) (at 97.028 94.234 0)
       (effects (font (size 1.27 1.27)) hide)
     )
@@
   (symbol (lib_id "power:GND") (at 171.958 71.374 0) (unit 1)
     (in_bom yes) (on_board yes) (fields_autoplaced)
-    (property "Reference" "#PWR014" (id 0) (at 171.958 77.724 0)
+    (property "Reference" "#PWR013" (id 0) (at 171.958 77.724 0)
       (effects (font (size 1.27 1.27)) hide)
     )
@@
   (symbol (lib_id "power:GND") (at 171.958 55.118 0) (unit 1)
     (in_bom yes) (on_board yes) (fields_autoplaced)
-    (property "Reference" "#PWR013" (id 0) (at 171.958 61.468 0)
+    (property "Reference" "#PWR012" (id 0) (at 171.958 61.468 0)
       (effects (font (size 1.27 1.27)) hide)
     )
@@
   (symbol (lib_id "power:GND") (at 171.958 103.886 0) (unit 1)
     (in_bom yes) (on_board yes) (fields_autoplaced)
-    (property "Reference" "#PWR016" (id 0) (at 171.958 110.236 0)
+    (property "Reference" "#PWR015" (id 0) (at 171.958 110.236 0)
       (effects (font (size 1.27 1.27)) hide)
     )
@@
   (symbol (lib_id "power:GND") (at 138.43 112.268 0) (unit 1)
     (in_bom yes) (on_board yes) (fields_autoplaced)
-    (property "Reference" "#PWR012" (id 0) (at 138.43 118.618 0)
+    (property "Reference" "#PWR011" (id 0) (at 138.43 118.618 0)
       (effects (font (size 1.27 1.27)) hide)
     )
@@
   (symbol (lib_id "power:GND") (at 171.958 87.63 0) (unit 1)
     (in_bom yes) (on_board yes) (fields_autoplaced)
-    (property "Reference" "#PWR015" (id 0) (at 171.958 93.98 0)
-      (effects (font (size 1.27 1.27)) hide)
-    )
+    (property "Reference" "#PWR014" (id 0) (at 171.958 93.98 0)
+      (effects (font (size 1.27 1.27)) hide)
+    )

Commit message: Mosfet crazy town
Parts:
- renumbered C2 to C3, C3 to C4, C4 to C5, C5 to C6, C6 to C7, U2 to U3
Changed lines of the file:
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@@
   (symbol (lib_id "Device:C") (at 138.43 105.156 0) (unit 1)
     (in_bom yes) (on_board yes) (fields_autoplaced)
-    (property "Reference" "C6" (id 0) (at 142.24 103.8859 0)
+    (property "Reference" "C7" (id 0) (at 142.24 103.8859 0)
       (effects (font (size 1.27 1.27)) (justify left))
     )
@@
   (symbol (lib_id "power:GND") (at 112.014 83.566 0) (unit 1)
     (in_bom yes) (on_board yes) (fields_autoplaced)
-    (property "Reference" "#PWR010" (id 0) (at 112.014 89.916 0)
+    (property "Reference" "#PWR015" (id 0) (at 112.014 89.916 0)
       (effects (font (size 1.27 1.27)) hide)
     )
@@
   (symbol (lib_id "74xx:74HC165") (at 97.028 61.976 0) (mirror y) (unit 1)
     (in_bom yes) (on_board yes) (fields_autoplaced)
-    (property "Reference" "U2" (id 0) (at 97.5486 39.116 0)
+    (property "Reference" "U3" (id 0) (at 97.5486 39.116 0)
       (effects (font (size 1.27 1.27)) (justify right))
     )
@@
   (symbol (lib_id "Device:C") (at 137.922 55.626 0) (unit 1)
     (in_bom yes) (on_board yes) (fields_autoplaced)
-    (property "Reference" "C3" (id 0) (at 141.732 54.3559 0)
+    (property "Reference" "C4" (id 0) (at 141.732 54.3559 0)
       (effects (font (size 1.27 1.27)) (justify left))
     )
@@
   (symbol (lib_id "power:GND") (at 97.028 87.884 0) (unit 1)
     (in_bom yes) (on_board yes) (fields_autoplaced)
-    (property "Reference" "#PWR09" (id 0) (at 97.028 94.234 0)
+    (property "Reference" "#PWR014" (id 0) (at 97.028 94.234 0)
       (effects (font (size 1.27 1.27)) hide)
     )
@@
   (symbol (lib_id "Device:C") (at 137.922 87.884 0) (unit 1)
     (in_bom yes) (on_board yes) (fields_autoplaced)
-    (property "Reference" "C5" (id 0) (at 141.732 86.6139 0)
+    (property "Reference" "C6" (id 0) (at 141.732 86.6139 0)
       (effects (font (size 1.27 1.27)) (justify left))
     )
@@
   (symbol (lib_id "Device:C") (at 61.976 48.006 0) (unit 1)
     (in_bom yes) (on_board yes) (fields_autoplaced)
-    (property "Reference" "C2" (id 0) (at 65.786 46.7359 0)
+    (property "Reference" "C3" (id 0) (at 65.786 46.7359 0)
       (effects (font (size 1.27 1.27)) (justify left))
     )
@@
   (symbol (lib_id "power:GND") (at 171.958 71.374 0) (unit 1)
     (in_bom yes) (on_board yes) (fields_autoplaced)
-    (property "Reference" "#PWR013" (id 0) (at 171.958 77.724 0)
+    (property "Reference" "#PWR018" (id 0) (at 171.958 77.724 0)
       (effects (font (size 1.27 1.27)) hide)
     )
@@
   (symbol (lib_id "power:GND") (at 171.958 55.118 0) (unit 1)
     (in_bom yes) (on_board yes) (fields_autoplaced)
-    (property "Reference" "#PWR012" (id 0) (at 171.958 61.468 0)
+    (property "Reference" "#PWR017" (id 0) (at 171.958 61.468 0)
       (effects (font (size 1.27 1.27)) hide)
     )
@@
   (symbol (lib_id "power:GND") (at 171.958 103.886 0) (unit 1)
     (in_bom yes) (on_board yes) (fields_autoplaced)
-    (property "Reference" "#PWR015" (id 0) (at 171.958 110.236 0)
+    (property "Reference" "#PWR020" (id 0) (at 171.958 110.236 0)
       (effects (font (size 1.27 1.27)) hide)
     )
@@
   (symbol (lib_id "Device:C") (at 137.922 71.882 0) (unit 1)
     (in_bom yes) (on_board yes) (fields_autoplaced)
-    (property "Reference" "C4" (id 0) (at 141.732 70.6119 0)
+    (property "Reference" "C5" (id 0) (at 141.732 70.6119 0)
       (effects (font (size 1.27 1.27)) (justify left))
     )
@@
   (symbol (lib_id "power:GND") (at 138.43 112.268 0) (unit 1)
     (in_bom yes) (on_board yes) (fields_autoplaced)
-    (property "Reference" "#PWR011" (id 0) (at 138.43 118.618 0)
+    (property "Reference" "#PWR016" (id 0) (at 138.43 118.618 0)
       (effects (font (size 1.27 1.27)) hide)
     )
@@
   (symbol (lib_id "power:GND") (at 171.958 87.63 0) (unit 1)
     (in_bom yes) (on_board yes) (fields_autoplaced)
-    (property "Reference" "#PWR014" (id 0) (at 171.958 93.98 0)
-      (effects (font (size 1.27 1.27)) hide)
-    )
+    (property "Reference" "#PWR019" (id 0) (at 171.958 93.98 0)
+      (effects (font (size 1.27 1.27)) hide)
+    )

Commit message: David FFS Merge pt 7
Parts:
- removed IC1, IC2, IC3, IC4: AH1902-Z-7, HallSensor:AH1902Z7, symbol AH1902-Z-7:AH1902-Z-7
- added U4, U5, U6, U7: SOT95, SOT95:SOT95P230X110-3N, symbol Sensor_Magnetic:A1101ELHL
- C3: LCSC (none) -> C15850
- C4, C5, C6, C7: LCSC (none) -> C1525
- U3: LCSC (none) -> C5613
Connections:
- net 3V: now also U4.1 (VCC), U5.1 (VCC), U6.1 (VCC), U7.1 (VCC)
- net GND: now also U4.3 (GND), U5.3 (GND), U6.3 (GND), U7.3 (GND)
- net at U3.11 (D0): now also U5.2 (VOUT)
- net at U3.12 (D1): now also U6.2 (VOUT)
- net at U3.13 (D2): now also U4.2 (VOUT)
- net at U3.14 (D3): now also U7.2 (VOUT)
Other:
- company: (none) -> Rowdy Chess
- title: (none) -> Rowdy Test Board
