File: KiCad Files/coils.kicad_sch (KiCad schematic)
At the start: 28 parts, among them Q1 AO3400A, Q10 AO3400A, Q11 AO3400A, Q12 AO3400A, Q13 AO3401A, Q14 AO3401A, Q15 AO3401A, Q16 AO3401A, Q2 AO3400A, Q3 AO3400A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

Commit message: Final pt 1
Other:
- note added: "Coil 1"
- note added: "Coil 10"
- note added: "Coil 11"
- note added: "Coil 12"
- note added: "Coil 13"
- note added: "Coil 14"
- note added: "Coil 15"
- note added: "Coil 16"
- note added: "Coil 2"
- note added: "Coil 3"
- note added: "Coil 4"
- note added: "Coil 5"
- note added: "Coil 6"
- note added: "Coil 7"
- note added: "Coil 8"
- note added: "Coil 9"
- note added: "Coil Shift Register"
- note added: "Ground Coils"
- note added: "Power Coils"
- note added: "Reverse Coil Shift Register"
- note added: "Reverse Ground Coils"
- note added: "Reverse Power Coils"
- company: (none) -> Rowdy Chess
- title: (none) -> Rowdy Test Board

Commit message: Generated JLC PCB Files
Parts:
- C1, C2: LCSC (none) -> C15850
- Q1, Q10, Q11, Q12, Q2, Q3, Q4, Q9: LCSC (none) -> C20917
- Q13, Q14, Q15, Q16, Q5, Q6, Q7, Q8: LCSC (none) -> C15127
- R1, R2, R3, R4, R5, R6, R7, R8: LCSC (none) -> C25804
- U1, U2: LCSC (none) -> C5947
Changed lines of the file:
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@@
+      (effects (font (size 1.27 1.27)) hide)
+    )
+    (property "LCSC" "C15127" (id 5) (at 211.328 68.326 0)
       (effects (font (size 1.27 1.27)) hide)
     )
@@
     )
     (property "JLC Part Number" "C15127" (id 4) (at 211.328 101.092 0)
+      (effects (font (size 1.27 1.27)) hide)
+    )
+    (property "LCSC" "C15127" (id 5) (at 211.328 101.092 0)
       (effects (font (size 1.27 1.27)) hide)
     )
@@
       (effects (font (size 1.27 1.27)) hide)
     )
+    (property "LCSC" "C15127" (id 5) (at 211.328 52.324 0)
+      (effects (font (size 1.27 1.27)) hide)
+    )
     (pin "1")
     (pin "2")
@@
       (effects (font (size 1.27 1.27)) hide)
     )
+    (property "LCSC" "C25804" (id 5) (at 123.952 28.448 0)
+      (effects (font (size 1.27 1.27)) hide)
+    )
     (pin "1")
     (pin "2")
@@
       (effects (font (size 1.27 1.27)) hide)
     )
+    (property "LCSC" "C15127" (id 5) (at 152.146 33.528 0)
+      (effects (font (size 1.27 1.27)) hide)
+    )
     (pin "1")
     (pin "2")
@@
     )
     (property "JLC Part Number" "C5947" (id 4) (at 250.952 139.7 0)
+      (effects (font (size 1.27 1.27)) hide)
+    )
+    (property "LCSC" "C5947" (id 5) (at 250.952 139.7 0)
       (effects (font (size 1.27 1.27)) hide)
     )
@@
       (effects (font (size 1.27 1.27)) hide)
     )
+    (property "LCSC" "C25804" (id 5) (at 186.182 28.448 0)
+      (effects (font (size 1.27 1.27)) hide)
+    )
     (pin "1")
     (pin "2")
@@
       (effects (font (size 1.27 1.27)) hide)
     )
+    (property "LCSC" "C20917" (id 5) (at 156.972 120.142 0)
+      (effects (font (size 1.27 1.27)) hide)
+    )
     (pin "1")
     (pin "2")
@@
       (effects (font (size 1.27 1.27)) hide)
     )
+    (property "LCSC" "C15850" (id 5) (at 281.686 136.652 0)
+      (effects (font (size 1.27 1.27)) hide)
+    )
     (pin "1")
     (pin "2")
@@
     )
     (property "JLC Part Number" "C20917" (id 4) (at 105.41 95.758 0)
+      (effects (font (size 1.27 1.27)) hide)
+    )
+    (property "LCSC" "C20917" (id 5) (at 105.41 95.758 0)
       (effects (font (size 1.27 1.27)) hide)
     )
@@
       (effects (font (size 1.27 1.27)) hide)
     )
+    (property "LCSC" "C20917" (id 5) (at 105.41 79.248 0)
+      (effects (font (size 1.27 1.27)) hide)
+    )
     (pin "1")
     (pin "2")
@@
       (effects (font (size 1.27 1.27)) hide)
     )
+    (property "LCSC" "C25804" (id 5) (at 216.408 60.452 0)
+      (effects (font (size 1.27 1.27)) hide)
+    )
     (pin "1")
     (pin "2")
@@
     )
     (property "JLC Part Number" "C5947" (id 4) (at 46.482 43.688 0)
+      (effects (font (size 1.27 1.27)) hide)
+    )
+    (property "LCSC" "C5947" (id 5) (at 46.482 43.688 0)
       (effects (font (size 1.27 1.27)) hide)
     )
@@
       (effects (font (size 1.27 1.27)) hide)
     )
+    (property "LCSC" "C25804" (id 5) (at 216.408 76.708 0)
+      (effects (font (size 1.27 1.27)) hide)
+    )
     (pin "1")
     (pin "2")
@@
       (effects (font (size 1.27 1.27)) hide)
     )
+    (property "LCSC" "C20917" (id 5) (at 105.41 62.738 0)
+      (effects (font (size 1.27 1.27)) hide)
+    )
     (pin "1")
     (pin "2")
@@
       (effects (font (size 1.27 1.27)) hide)
     )
+    (property "LCSC" "C20917" (id 5) (at 105.41 112.268 0)
+      (effects (font (size 1.27 1.27)) hide)
+    )
     (pin "1")
     (pin "2")
@@
       (effects (font (size 1.27 1.27)) hide)
     )
+    (property "LCSC" "C25804" (id 5) (at 144.272 28.448 0)
+      (effects (font (size 1.27 1.27)) hide)
+    )
     (pin "1")
     (pin "2")
@@
     )
     (property "JLC Part Number" "C15127" (id 4) (at 211.328 84.582 0)
+      (effects (font (size 1.27 1.27)) hide)
+    )
+    (property "LCSC" "C15127" (id 5) (at 211.328 84.582 0)
       (effects (font (size 1.27 1.27)) hide)
     )
@@
       (effects (font (size 1.27 1.27)) hide)
     )
+    (property "LCSC" "C25804" (id 5) (at 216.408 44.45 0)
+      (effects (font (size 1.27 1.27)) hide)
+    )
     (pin "1")
     (pin "2")
@@
       (effects (font (size 1.27 1.27)) hide)
     )
+    (property "LCSC" "C25804" (id 5) (at 165.608 28.448 0)
+      (effects (font (size 1.27 1.27)) hide)
+    )
     (pin "1")
     (pin "2")
@@
       (effects (font (size 1.27 1.27)) hide)
     )
+    (property "LCSC" "C25804" (id 5) (at 216.408 93.218 0)
+      (effects (font (size 1.27 1.27)) hide)
+    )
     (pin "1")
     (pin "2")
@@
       (effects (font (size 1.27 1.27)) hide)
     )
+    (property "LCSC" "C15127" (id 5) (at 131.826 33.528 0)
+      (effects (font (size 1.27 1.27)) hide)
+    )
     (pin "1")
     (pin "2")
@@
       (effects (font (size 1.27 1.27)) hide)
     )
+    (property "LCSC" "C15127" (id 5) (at 173.482 33.528 0)
+      (effects (font (size 1.27 1.27)) hide)
+    )
     (pin "1")
     (pin "2")
@@
       (effects (font (size 1.27 1.27)) hide)
     )
+    (property "LCSC" "C15127" (id 5) (at 194.056 33.528 0)
+      (effects (font (size 1.27 1.27)) hide)
+    )
     (pin "1")
     (pin "2")
@@
       (effects (font (size 1.27 1.27)) hide)
     )
+    (property "LCSC" "C20917" (id 5) (at 136.652 120.142 0)
+      (effects (font (size 1.27 1.27)) hide)
+    )
     (pin "1")
     (pin "2")
@@
     )
     (property "JLC Part Number" "C15850" (id 4) (at 15.748 40.64 0)
+      (effects (font (size 1.27 1.27)) hide)
+    )
+    (property "LCSC" "C15850" (id 5) (at 15.748 40.64 0)
       (effects (font (size 1.27 1.27)) hide)
     )
@@
       (effects (font (size 1.27 1.27)) hide)
     )
+    (property "LCSC" "C20917" (id 5) (at 198.882 120.142 0)
+      (effects (font (size 1.27 1.27)) hide)
+    )
     (pin "1")
     (pin "2")
@@
       (effects (font (size 1.27 1.27)) hide)
     )
+    (property "LCSC" "C20917" (id 5) (at 178.308 120.142 0)
+      (effects (font (size 1.27 1.27)) hide)
+    )
