File: KiCad Files/coils.kicad_sch (KiCad schematic)
At the start: 13 parts, among them Q1 AO3400A, Q2 AO3400A, Q3 AO3400A, Q4 AO3400A, Q5 AO3401A, Q6 AO3401A, Q7 AO3401A, Q8 AO3401A, U2 74HC595

Commit message: Business
Connections:
- net at Q1.3 (D), Q2.3 (D), Q3.3 (D)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: no longer Q7.1 (G), R3.2, U2.2 (QC)
- new net: Q7.1 (G), R3.2, U2.2 (QC)
Changed lines of the file:
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@@
   (junction (at 198.882 35.052) (diameter 0) (color 0 0 0 0)
   )
-  (junction (at 167.386 51.308) (diameter 0) (color 0 0 0 0)
-  )
   (junction (at 188.722 35.052) (diameter 0) (color 0 0 0 0)
   )
@@
   (junction (at 191.516 87.884) (diameter 0) (color 0 0 0 0)
   )
-  (junction (at 147.066 51.308) (diameter 0) (color 0 0 0 0)
-  )
   (junction (at 136.652 35.052) (diameter 0) (color 0 0 0 0)
   )
@@
     (stroke (width 0) (type default) (color 0 0 0 0))
   )
+  (wire (pts (xy 69.342 51.816) (xy 69.342 51.308))
+    (stroke (width 0) (type default) (color 0 0 0 0))
+  )
   (wire (pts (xy 69.342 56.388) (xy 113.03 56.388))
     (stroke (width 0) (type default) (color 0 0 0 0))
@@
     (stroke (width 0) (type default) (color 0 0 0 0))
   )
-  (wire (pts (xy 147.066 51.308) (xy 167.386 51.308))
+  (wire (pts (xy 69.342 51.816) (xy 181.102 51.816))
     (stroke (width 0) (type default) (color 0 0 0 0))
   )
@@
     (stroke (width 0) (type default) (color 0 0 0 0))
   )
-  (wire (pts (xy 69.342 51.308) (xy 147.066 51.308))
-    (stroke (width 0) (type default) (color 0 0 0 0))
-  )
   (wire (pts (xy 170.18 104.648) (xy 167.386 104.648))
     (stroke (width 0) (type default) (color 0 0 0 0))
@@
     (stroke (width 0) (type default) (color 0 0 0 0))
   )
-  (wire (pts (xy 167.386 51.308) (xy 181.102 51.308))
-    (stroke (width 0) (type default) (color 0 0 0 0))
-  )
   (wire (pts (xy 167.386 103.378) (xy 188.722 103.378))
     (stroke (width 0) (type default) (color 0 0 0 0))
@@
     (stroke (width 0) (type default) (color 0 0 0 0))
   )
-  (wire (pts (xy 181.102 46.228) (xy 181.102 51.308))
-    (stroke (width 0) (type default) (color 0 0 0 0))
-  )
+  (wire (pts (xy 181.102 46.228) (xy 181.102 51.816))
+    (stroke (width 0) (type default) (color 0 0 0 0))
+  )

Commit message: Big saucy business
Parts:
- added C1: 10u, Capacitor_SMD:C_0805_2012Metric, symbol Device:C
Connections:
- net 5V: now also C1.1; no longer Q5.2 (S), Q6.2 (S), Q7.2 (S), Q8.2 (S), R1.1, R2.1, R3.1, R4.1
- net GND: now also C1.2
- new net Vbus: Q5.2 (S), Q6.2 (S), Q7.2 (S), Q8.2 (S), R1.1, R2.1, R3.1, R4.1
Changed lines of the file:
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@@
   (junction (at 191.516 87.884) (diameter 0) (color 0 0 0 0)
   )
+  (junction (at 188.722 119.888) (diameter 0) (color 0 0 0 0)
+  )
+  (junction (at 188.722 54.864) (diameter 0) (color 0 0 0 0)
+  )
+  (junction (at 201.676 46.228) (diameter 0) (color 0 0 0 0)
+  )
+  (junction (at 188.722 70.358) (diameter 0) (color 0 0 0 0)
+  )
+  (junction (at 149.86 88.138) (diameter 0) (color 0 0 0 0)
+  )
+  (junction (at 167.386 55.118) (diameter 0) (color 0 0 0 0)
+  )
+  (junction (at 59.182 74.676) (diameter 0) (color 0 0 0 0)
+  )
+  (junction (at 181.102 46.228) (diameter 0) (color 0 0 0 0)
+  )
+  (junction (at 170.18 71.628) (diameter 0) (color 0 0 0 0)
+  )
+  (junction (at 167.386 35.052) (diameter 0) (color 0 0 0 0)
+  )
   (junction (at 136.652 35.052) (diameter 0) (color 0 0 0 0)
   )
-  (junction (at 188.722 119.888) (diameter 0) (color 0 0 0 0)
-  )
-  (junction (at 188.722 54.864) (diameter 0) (color 0 0 0 0)
-  )
-  (junction (at 201.676 46.228) (diameter 0) (color 0 0 0 0)
-  )
-  (junction (at 188.722 70.358) (diameter 0) (color 0 0 0 0)
-  )
-  (junction (at 149.86 88.138) (diameter 0) (color 0 0 0 0)
-  )
-  (junction (at 132.08 35.052) (diameter 0) (color 0 0 0 0)
-  )
-  (junction (at 167.386 55.118) (diameter 0) (color 0 0 0 0)
-  )
-  (junction (at 181.102 46.228) (diameter 0) (color 0 0 0 0)
-  )
-  (junction (at 170.18 71.628) (diameter 0) (color 0 0 0 0)
-  )
-  (junction (at 167.386 35.052) (diameter 0) (color 0 0 0 0)
-  )
   (junction (at 209.296 54.864) (diameter 0) (color 0 0 0 0)
   )
@@
   (junction (at 147.066 103.378) (diameter 0) (color 0 0 0 0)
   )
+  (junction (at 59.182 37.338) (diameter 0) (color 0 0 0 0)
+  )
   (junction (at 178.308 35.052) (diameter 0) (color 0 0 0 0)
   )
@@
     (stroke (width 0) (type default) (color 0 0 0 0))
   )
+  (wire (pts (xy 28.448 49.53) (xy 28.448 37.338))
+    (stroke (width 0) (type default) (color 0 0 0 0))
+  )
   (wire (pts (xy 198.882 44.958) (xy 198.882 46.228))
     (stroke (width 0) (type default) (color 0 0 0 0))
@@
     (stroke (width 0) (type default) (color 0 0 0 0))
   )
-  (wire (pts (xy 59.182 35.052) (xy 59.182 41.148))
+  (wire (pts (xy 59.182 33.02) (xy 59.182 37.338))
     (stroke (width 0) (type default) (color 0 0 0 0))
   )
@@
     (stroke (width 0) (type default) (color 0 0 0 0))
   )
+  (wire (pts (xy 136.398 35.052) (xy 136.652 35.052))
+    (stroke (width 0) (type default) (color 0 0 0 0))
+  )
   (wire (pts (xy 136.652 46.228) (xy 139.446 46.228))
     (stroke (width 0) (type default) (color 0 0 0 0))
@@
     (stroke (width 0) (type default) (color 0 0 0 0))
   )
+  (wire (pts (xy 136.398 29.21) (xy 136.398 35.052))
+    (stroke (width 0) (type default) (color 0 0 0 0))
+  )
   (wire (pts (xy 149.86 104.648) (xy 149.86 88.138))
     (stroke (width 0) (type default) (color 0 0 0 0))
@@
     (stroke (width 0) (type default) (color 0 0 0 0))
   )
-  (wire (pts (xy 132.08 35.052) (xy 136.652 35.052))
-    (stroke (width 0) (type default) (color 0 0 0 0))
-  )
   (wire (pts (xy 212.09 71.374) (xy 209.296 71.374))
     (stroke (width 0) (type default) (color 0 0 0 0))
@@
     (stroke (width 0) (type default) (color 0 0 0 0))
   )
+  (wire (pts (xy 59.182 37.338) (xy 59.182 41.148))
+    (stroke (width 0) (type default) (color 0 0 0 0))
+  )
   (wire (pts (xy 191.516 104.394) (xy 191.516 87.884))
     (stroke (width 0) (type default) (color 0 0 0 0))
@@
     (stroke (width 0) (type default) (color 0 0 0 0))
   )
+  (wire (pts (xy 59.182 74.676) (xy 59.182 74.93))
+    (stroke (width 0) (type default) (color 0 0 0 0))
+  )
   (wire (pts (xy 113.03 108.458) (xy 107.95 108.458))
     (stroke (width 0) (type default) (color 0 0 0 0))
@@
     (stroke (width 0) (type default) (color 0 0 0 0))
   )
+  (wire (pts (xy 28.448 37.338) (xy 59.182 37.338))
+    (stroke (width 0) (type default) (color 0 0 0 0))
+  )
   (wire (pts (xy 170.18 88.138) (xy 170.18 71.628))
     (stroke (width 0) (type default) (color 0 0 0 0))
@@
     (stroke (width 0) (type default) (color 0 0 0 0))
   )
+  (wire (pts (xy 59.182 74.168) (xy 59.182 74.676))
+    (stroke (width 0) (type default) (color 0 0 0 0))
+  )
   (wire (pts (xy 107.95 61.468) (xy 69.342 61.468))
     (stroke (width 0) (type default) (color 0 0 0 0))
@@
     (stroke (width 0) (type default) (color 0 0 0 0))
   )
-  (wire (pts (xy 59.182 35.052) (xy 132.08 35.052))
-    (stroke (width 0) (type default) (color 0 0 0 0))
-  )
   (wire (pts (xy 212.09 71.374) (xy 212.09 54.864))
     (stroke (width 0) (type default) (color 0 0 0 0))
@@
     (stroke (width 0) (type default) (color 0 0 0 0))
   )
+  (wire (pts (xy 28.448 57.15) (xy 28.448 74.676))
+    (stroke (width 0) (type default) (color 0 0 0 0))
+  )
   (wire (pts (xy 209.296 51.308) (xy 209.296 54.864))
     (stroke (width 0) (type default) (color 0 0 0 0))
@@
     (stroke (width 0) (type default) (color 0 0 0 0))
   )
-  (wire (pts (xy 132.08 33.02) (xy 132.08 35.052))
+  (wire (pts (xy 28.448 74.676) (xy 59.182 74.676))
     (stroke (width 0) (type default) (color 0 0 0 0))
   )
@@
     (effects (font (size 1.27 1.27)) (justify left))
   )
-  (hierarchical_label "5V" (shape input) (at 132.08 33.02 180)
+  (hierarchical_label "5V" (shape input) (at 59.182 33.02 180)
     (effects (font (size 1.27 1.27)) (justify right))
   )
@@
     (effects (font (size 1.27 1.27)) (justify right))
   )
+  (hierarchical_label "Vbus" (shape input) (at 136.398 29.21 180)
+    (effects (font (size 1.27 1.27)) (justify right))
+  )
   (symbol (lib_id "Device:R") (at 136.652 41.148 0) (unit 1)
     (in_bom yes) (on_board yes) (fields_autoplaced)
@@
   (symbol (lib_id "power:GND") (at 120.65 97.028 0) (unit 1)
     (in_bom yes) (on_board yes) (fields_autoplaced)
-    (property "Reference" "#PWR04" (id 0) (at 120.65 103.378 0)
+    (property "Reference" "#PWR07" (id 0) (at 120.65 103.378 0)
       (effects (font (size 1.27 1.27)) hide)
     )
@@
   (symbol (lib_id "power:GND") (at 120.65 130.048 0) (unit 1)
     (in_bom yes) (on_board yes) (fields_autoplaced)
-    (property "Reference" "#PWR06" (id 0) (at 120.65 136.398 0)
+    (property "Reference" "#PWR09" (id 0) (at 120.65 136.398 0)
       (effects (font (size 1.27 1.27)) hide)
     )
@@
   (symbol (lib_id "power:GND") (at 120.65 80.518 0) (unit 1)
     (in_bom yes) (on_board yes) (fields_autoplaced)
-    (property "Reference" "#PWR03" (id 0) (at 120.65 86.868 0)
+    (property "Reference" "#PWR06" (id 0) (at 120.65 86.868 0)
       (effects (font (size 1.27 1.27)) hide)
     )
@@
     (pin "3")
   )
-  (symbol (lib_id "power:GND") (at 59.182 74.168 0) (unit 1)
-    (in_bom yes) (on_board yes) (fields_autoplaced)
-    (property "Reference" "#PWR02" (id 0) (at 59.182 80.518 0)
-      (effects (font (size 1.27 1.27)) hide)
-    )
-    (property "Value" "GND" (id 1) (at 59.182 78.74 0))
-    (property "Footprint" "" (id 2) (at 59.182 74.168 0)
-      (effects (font (size 1.27 1.27)) hide)
-    )
-    (property "Datasheet" "" (id 3) (at 59.182 74.168 0)
+  (symbol (lib_id "Device:C") (at 28.448 53.34 0) (unit 1)
+    (in_bom yes) (on_board yes) (fields_autoplaced)
+    (property "Reference" "C1" (id 0) (at 32.258 52.0699 0)
+      (effects (font (size 1.27 1.27)) (justify left))
+    )
+    (property "Value" "10u" (id 1) (at 32.258 54.6099 0)
+      (effects (font (size 1.27 1.27)) (justify left))
+    )
+    (property "Footprint" "Capacitor_SMD:C_0805_2012Metric" (id 2) (at 29.4132 57.15 0)
+      (effects (font (size 1.27 1.27)) hide)
+    )
+    (property "Datasheet" "https://datasheet.lcsc.com/lcsc/1811121310_Samsung-Electro-Mechanics-CL21A106KAYNNNE_C15850.pdf" (id 3) (at 28.448 53.34 0)
+      (effects (font (size 1.27 1.27)) hide)
+    )
+    (property "JLC Part Number" "C15850" (id 4) (at 28.448 53.34 0)
+      (effects (font (size 1.27 1.27)) hide)
+    )
+    (pin "1")
+    (pin "2")
+  )
+  (symbol (lib_id "power:GND") (at 59.182 74.93 0) (unit 1)
+    (in_bom yes) (on_board yes) (fields_autoplaced)
+    (property "Reference" "#PWR05" (id 0) (at 59.182 81.28 0)
+      (effects (font (size 1.27 1.27)) hide)
+    )
+    (property "Value" "GND" (id 1) (at 59.182 79.502 0))
+    (property "Footprint" "" (id 2) (at 59.182 74.93 0)
+      (effects (font (size 1.27 1.27)) hide)
+    )
+    (property "Datasheet" "" (id 3) (at 59.182 74.93 0)
       (effects (font (size 1.27 1.27)) hide)
     )
@@
   (symbol (lib_id "power:GND") (at 120.65 113.538 0) (unit 1)
     (in_bom yes) (on_board yes) (fields_autoplaced)
-    (property "Reference" "#PWR05" (id 0) (at 120.65 119.888 0)
-      (effects (font (size 1.27 1.27)) hide)
-    )
+    (property "Reference" "#PWR08" (id 0) (at 120.65 119.888 0)
+      (effects (font (size 1.27 1.27)) hide)
+    )

Commit message: Big coils baby
Parts:
- renumbered U2 to U1
Changed lines of the file:
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@@
   (symbol (lib_id "power:GND") (at 120.65 97.028 0) (unit 1)
     (in_bom yes) (on_board yes) (fields_autoplaced)
-    (property "Reference" "#PWR07" (id 0) (at 120.65 103.378 0)
+    (property "Reference" "#PWR06" (id 0) (at 120.65 103.378 0)
       (effects (font (size 1.27 1.27)) hide)
     )
@@
   (symbol (lib_id "74xx:74HC595") (at 59.182 56.388 0) (unit 1)
     (in_bom yes) (on_board yes)
-    (property "Reference" "U2" (id 0) (at 61.2014 38.354 0)
+    (property "Reference" "U1" (id 0) (at 61.2014 38.354 0)
       (effects (font (size 1.27 1.27)) (justify left))
     )
@@
   (symbol (lib_id "power:GND") (at 120.65 130.048 0) (unit 1)
     (in_bom yes) (on_board yes) (fields_autoplaced)
-    (property "Reference" "#PWR09" (id 0) (at 120.65 136.398 0)
+    (property "Reference" "#PWR08" (id 0) (at 120.65 136.398 0)
       (effects (font (size 1.27 1.27)) hide)
     )
@@
   (symbol (lib_id "power:GND") (at 120.65 80.518 0) (unit 1)
     (in_bom yes) (on_board yes) (fields_autoplaced)
-    (property "Reference" "#PWR06" (id 0) (at 120.65 86.868 0)
+    (property "Reference" "#PWR05" (id 0) (at 120.65 86.868 0)
       (effects (font (size 1.27 1.27)) hide)
     )
@@
   (symbol (lib_id "power:GND") (at 59.182 74.93 0) (unit 1)
     (in_bom yes) (on_board yes) (fields_autoplaced)
-    (property "Reference" "#PWR05" (id 0) (at 59.182 81.28 0)
+    (property "Reference" "#PWR04" (id 0) (at 59.182 81.28 0)
       (effects (font (size 1.27 1.27)) hide)
     )
@@
   (symbol (lib_id "power:GND") (at 120.65 113.538 0) (unit 1)
     (in_bom yes) (on_board yes) (fields_autoplaced)
-    (property "Reference" "#PWR08" (id 0) (at 120.65 119.888 0)
-      (effects (font (size 1.27 1.27)) hide)
-    )
+    (property "Reference" "#PWR07" (id 0) (at 120.65 119.888 0)
+      (effects (font (size 1.27 1.27)) hide)
+    )

Commit message: Mosfet crazy town
Parts:
- added C2: 10u, Capacitor_SMD:C_0805_2012Metric, symbol Device:C
- added Q10, Q11, Q12, Q9: AO3400A, Package_TO_SOT_SMD:SOT-23, symbol Transistor_FET:AO3400A
- added Q13, Q14, Q15, Q16: AO3401A, Package_TO_SOT_SMD:SOT-23, symbol Transistor_FET:AO3401A
- added R5, R6, R7, R8: 10K, Resistor_SMD:R_0603_1608Metric, symbol Device:R
- added U2: 74HC595, 74HC595:SO16, symbol 74xx:74HC595
Connections:
- net 5V: now also C2.1, U2.16 (VCC)
- net GND: now also C2.2, Q10.2 (S), Q11.2 (S), Q12.2 (S), Q9.2 (S), U2.8 (GND)
- net NMR: now also U2.10 (~{SRCLR})
- net NOE: now also U2.13 (~{OE})
- net QH': now also U2.9 (QH'); no longer U1.9 (QH')
- net SHCP: now also U2.11 (SRCLK)
- net STCP: now also U2.12 (RCLK)
- net Vbus: now also Q13.2 (S), Q14.2 (S), Q15.2 (S), Q16.2 (S), R5.1, R6.1, R7.1, R8.1
- net at Q1.3 (D), Q2.3 (D), Q3.3 (D)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: now also Q10.3 (D), Q11.3 (D), Q12.3 (D), Q13.3 (D), Q14.3 (D), Q15.3 (D), Q16.3 (D), Q9.3 (D)
- new net: Q14.1 (G), R6.2, U2.1 (QB)
- new net: Q16.1 (G), R8.2, U2.3 (QD)
- new net: Q13.1 (G), R5.2, U2.15 (QA)
- new net: U1.9 (QH'), U2.14 (SER)
- new net: Q15.1 (G), R7.2, U2.2 (QC)
- new net: Q9.1 (G), U2.4 (QE)
- new net: Q10.1 (G), U2.5 (QF)
- new net: Q11.1 (G), U2.6 (QG)
- new net: Q12.1 (G), U2.7 (QH)
Other:
- moved on the sheet: C1, Q1, Q2, Q3, Q4, Q5, Q6, Q7, Q8, R1, R2, R3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

Commit message: David FFS Merge pt 1
Parts:
- C1, C2: LCSC (none) -> C15850
- Q1, Q10, Q11, Q12, Q2, Q3, Q4, Q9: LCSC (none) -> C20917
- Q13, Q14, Q15, Q16, Q5, Q6, Q7, Q8: LCSC (none) -> C15127
- R1, R2, R3, R4, R5, R6, R7, R8: LCSC (none) -> C25804
- U1, U2: LCSC (none) -> C5947
Other:
- note added: "Coil 1"
- note added: "Coil 10"
- note added: "Coil 11"
- note added: "Coil 12"
- note added: "Coil 13"
- note added: "Coil 14"
- note added: "Coil 15"
- note added: "Coil 16"
- note added: "Coil 2"
- note added: "Coil 3"
- note added: "Coil 4"
- note added: "Coil 5"
- note added: "Coil 6"
- note added: "Coil 7"
- note added: "Coil 8"
- note added: "Coil 9"
- note added: "Coil Shift Register"
- note added: "Ground Coils"
- note added: "Power Coils"
- note added: "Reverse Coil Shift Register"
- note added: "Reverse Ground Coils"
- note added: "Reverse Power Coils"
- company: (none) -> Rowdy Chess
- title: (none) -> Rowdy Test Board
